File: Powerstage2/Powestage2.kicad_pcb (KiCad board)
At the start: 2 copper layers, 75.8 x 53.5 mm, 42 parts, among them J1 Conn_01x05_Female, Q1 BD139, Q2 BD140, Q3 BD139, Q4 BD140, Q5 C2M0025120D, Q6 C2M0025120D, U1 L7812, U2 U3115S

Commit message: Powerstage2 bearbeitet
Parts:
- removed Q1, Q3: BD139, Package_TO_SOT_THT:TO-126-3_Vertical
- removed Q2, Q4: BD140, Package_TO_SOT_THT:TO-126-3_Vertical
- added Q10: FZT953, Package_TO_SOT_SMD:SOT-223-3_TabPin2, F.Cu at (210.0, 97.0)
- added Q7: FZT853, Package_TO_SOT_SMD:SOT-223-3_TabPin2, F.Cu at (206.8, 123.0)
- added Q8: FZT953, Package_TO_SOT_SMD:SOT-223-3_TabPin2, F.Cu at (206.8, 131.0)
- added Q9: FZT853, Package_TO_SOT_SMD:SOT-223-3_TabPin2, F.Cu at (210.0, 89.0)
- moved R8 15.4 mm to (214.6, 102.2), turned to 180 degrees
- moved R4 9.41 mm to (195.0, 121.0), turned to 90 degrees
- moved C3 1.97 mm to (200.0, 124.0)
- moved R5 1.41 mm to (215.0, 84.0)
- moved D6 0.50 mm to (216.5, 88.5), turned to -90 degrees
Routing:
- net Net-(Q7-E): track 9.90 -> 23.6 mm
- net Net-(Q10-B): track 31.0 -> 20.8 mm, vias 1 -> 2
- net Net-(Q10-E): track 15.7 -> 23.3 mm, vias 0 -> 3
- net Net-(D6-A): track 91.4 -> 85.3 mm, vias 5 -> 4
- net Net-(U2-LO): track 30.8 -> 25.0 mm
- net Net-(D5-K): track 28.8 -> 33.3 mm
- net GND: track 47.2 -> 50.6 mm, vias 41 -> 47
- net +12V: track 130.2 -> 127.3 mm, vias 1 -> 0
- net Net-(Q7-B): track 22.9 -> 21.3 mm, vias 0 -> 2
- net Net-(D6-K): track 8.10 -> 8.98 mm
- net Net-(D3-A): track 44.5 -> 43.9 mm
Other:
- board text added: "Powerstage V4 2024_08_31"
- board text removed: "Powerstage V3 2021_01_06"
