File: Powerstage2/Powestage2.kicad_sch (KiCad schematic)
At the start: 42 parts, among them J1 Conn_01x05_Female, Q1 BD139, Q2 BD140, Q3 BD139, Q4 BD140, Q5 C2M0025120D, Q6 C2M0025120D, U1 L7812, U2 U3115S

Commit message: Powerstage2 bearbeitet
Parts:
- removed Q1, Q3: BD139, Package_TO_SOT_THT:TO-126-3_Vertical, symbol Transistor_BJT:BD139
- removed Q2, Q4: BD140, Package_TO_SOT_THT:TO-126-3_Vertical, symbol Transistor_BJT:BD140
- added Q10, Q8: FZT953, Package_TO_SOT_SMD:SOT-223-3_TabPin2, symbol Transistor_BJT:BCP51
- added Q7, Q9: FZT853, Package_TO_SOT_SMD:SOT-223-3_TabPin2, symbol Transistor_BJT:BCP56
Connections:
- net +12V: now also Q7.2 (C), Q7.4 (C)
- net GND: now also Q8.2 (C)
- net at D6.2 (A), H4.1, Q5.3 (S)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: now also Q10.2 (C)
- net at C9.1, D5.1 (K), U2.8 (VB): now also Q9.2 (C), Q9.4 (C)
- net at R3.1: now also Q10.1 (B), Q9.1 (B)
- net at R4.1: now also Q7.1 (B), Q8.1 (B)
- net at R5.2: now also Q10.3 (E), Q9.3 (E)
- net at R6.2: now also Q7.3 (E), Q8.3 (E)

Commit message: Kleinere Änderungen
Other:
- note added: "Anstatt R8 Diode bestücken, D3 und D4 kann dann entfallen."
- note added: "R7 und D8 für unterdrückung von Schwingungen, beide oder keine bestücken."
Changed lines of the file:
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@@
+		)
+	)
+	(text "Anstatt R8 Diode bestücken, D3 und D4 kann dann entfallen."
+		(exclude_from_sim no)
+		(at 226.06 124.46 0)
+		(effects
+			(font
+				(size 1.27 1.27)
+			)
+		)
+	)
+	(text "R7 und D8 für unterdrückung von Schwingungen, beide oder keine bestücken."
+		(exclude_from_sim no)
+		(at 233.68 128.27 0)
+		(effects
+			(font
+				(size 1.27 1.27)
+			)
 		)
 	)
