File: DCDC_mid/DCDC_mid.kicad_sch (KiCad schematic)
At the start: 36 parts, among them J1 Conn_01x02_Pin, J2 Conn_01x02_Pin, Q1 BD139, Q2 BD140, Q4 BD139, Q5 C2M0025120D, U1 LM311, U2 TL431LP

Commit message: DCDC_mit verbessert, hoffentlich
Parts:
- removed C7: 1u, Capacitor_SMD:C_0805_2012Metric_Pad1.18x1.45mm_HandSolder, symbol Device:C
- removed D4: D, Diode_SMD:D_SOD-123, symbol Device:D
- removed Q5: C2M0025120D, Package_TO_SOT_THT:TO-247-3_Vertical, symbol Transistor_FET:C2M0025120D
- added Q4: Q_PMOS_GDSD, Package_TO_SOT_SMD:TO-263-3_TabPin4, symbol Device:Q_PMOS_GDSD
- R7: renamed from R5; value 10R -> 1R
- renumbered C6 to C1, C5 to C2, C1 to C3, C9 to C4, C10 to C5, C2 to C6, C8 to C7, C3 to C8, C4 to C9, D2 to D1, D1 to D2, D5 to D3, D3 to D4, Q4 to Q1, Q1 to Q2, Q2 to Q3, R3 to R1, R1 to R3, R7 to R4, R6 to R5, R4 to R6, U2 to U1, U1 to U2
Connections:
- net +VDC: now also C7.2, Q2.2 (C), R6.1, Q4.3 (S)
- net at C3.1, R1.2, R2.1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: now also U2.2 (+); no longer U2.3 (-)
- net at C5.2, R4.1: now also U2.3 (-); no longer U2.2 (+)
- net at R7.2: now also Q4.1 (G)
- net at D3.1 (K), D4.1 (K), L1.1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: now also Q4.2 (D), Q4.4 (D)
Other:
- moved on the sheet: C5, R4

Commit message: DCDC_mid überarbeitet
Parts:
- added C10: 100n, Capacitor_SMD:C_0805_2012Metric_Pad1.18x1.45mm_HandSolder, symbol Device:C
- added R8: 13k, Resistor_SMD:R_0805_2012Metric_Pad1.20x1.40mm_HandSolder, symbol Device:R
Connections:
- net GND: now also C10.1
- net at C6.1, C8.1, C9.1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: now also R8.2; no longer R4.2
- new net: C10.2, R4.2, R8.1
Changed lines of the file:
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@@
 	(paper "A4")
 	(title_block
-		(date "2023-12-14")
+		(date "2024-08-17")
 		(rev "2")
-		(comment 1 "Inv und Nichtinv eingang vertauscht, Falscher footbrint für Leistungsdioden, RC-Glied in Rückkopplungsuzweig.")
+		(comment 1 "Falscher footbrint für Leistungsdioden")
+		(comment 2 "RC-Glied in Rückkopplungsuzweig")
+		(comment 3 "P-Kanal Mosfet ")
 	)
 	(junction
@@
 	)
 	(junction
+		(at 95.25 134.62)
+		(diameter 0)
+		(color 0 0 0 0)
+	)
+	(junction
 		(at 54.61 118.11)
 		(diameter 0)
@@
 	(wire
 		(pts
+			(xy 95.25 142.24) (xy 95.25 146.05)
+		)
+		(stroke
+			(width 0)
+			(type default)
+		)
+	)
+	(wire
+		(pts
 			(xy 46.99 74.93) (xy 50.8 74.93)
 		)
@@
 	(wire
 		(pts
+			(xy 95.25 134.62) (xy 102.87 134.62)
+		)
+		(stroke
+			(width 0)
+			(type default)
+		)
+	)
+	(wire
+		(pts
 			(xy 41.91 133.35) (xy 41.91 146.05)
 		)
@@
 	(wire
 		(pts
-			(xy 87.63 134.62) (xy 179.07 134.62)
+			(xy 87.63 134.62) (xy 95.25 134.62)
 		)
 		(stroke
@@
 	(wire
 		(pts
+			(xy 110.49 134.62) (xy 179.07 134.62)
+		)
+		(stroke
+			(width 0)
+			(type default)
+		)
+	)
+	(wire
+		(pts
 			(xy 132.08 105.41) (xy 132.08 111.76)
 		)
@@
 	)
 	(symbol
+		(lib_id "Device:R")
+		(at 106.68 134.62 90)
+		(unit 1)
+		(exclude_from_sim no)
+		(in_bom yes)
+		(on_board yes)
+		(dnp no)
+		(fields_autoplaced yes)
+		(property "Reference" "R8"
+			(at 106.68 128.27 90)
+			(effects
+				(font
+					(size 1.27 1.27)
+				)
+			)
+		)
+		(property "Value" "13k"
+			(at 106.68 130.81 90)
+			(effects
+				(font
+					(size 1.27 1.27)
+				)
+			)
+		)
+		(property "Footprint" "Resistor_SMD:R_0805_2012Metric_Pad1.20x1.40mm_HandSolder"
+			(at 106.68 136.398 90)
+			(effects
+				(font
+					(size 1.27 1.27)
+				)
+				(hide yes)
+			)
+		)
+		(property "Datasheet" "~"
+			(at 106.68 134.62 0)
+			(effects
+				(font
+					(size 1.27 1.27)
+				)
+				(hide yes)
+			)
+		)
+		(property "Description" ""
+			(at 106.68 134.62 0)
+			(effects
+				(font
+					(size 1.27 1.27)
+				)
+				(hide yes)
+			)
+		)
+		(pin "1"
+		)
+		(pin "2"
+		)
+		(instances
+			(project "DCDC_mid"
+				(path "/6223a5f4-c243-4547-8c88-bb7b5a32f283"
+					(reference "R8")
+					(unit 1)
+				)
+			)
+		)
+	)
+	(symbol
 		(lib_id "Device:L")
 		(at 137.16 111.76 90)
@@
 	)
 	(symbol
+		(lib_id "Device:C")
+		(at 95.25 138.43 180)
+		(unit 1)
+		(exclude_from_sim no)
+		(in_bom yes)
+		(on_board yes)
+		(dnp no)
+		(fields_autoplaced yes)
+		(property "Reference" "C10"
+			(at 99.06 137.1599 0)
+			(effects
+				(font
+					(size 1.27 1.27)
+				)
+				(justify right)
+			)
+		)
+		(property "Value" "100n"
+			(at 99.06 139.6999 0)
+			(effects
+				(font
+					(size 1.27 1.27)
+				)
+				(justify right)
+			)
+		)
+		(property "Footprint" "Capacitor_SMD:C_0805_2012Metric_Pad1.18x1.45mm_HandSolder"
+			(at 94.2848 134.62 0)
+			(effects
+				(font
+					(size 1.27 1.27)
+				)
+				(hide yes)
+			)
+		)
+		(property "Datasheet" "~"
+			(at 95.25 138.43 0)
+			(effects
+				(font
+					(size 1.27 1.27)
+				)
+				(hide yes)
+			)
+		)
+		(property "Description" ""
+			(at 95.25 138.43 0)
+			(effects
+				(font
+					(size 1.27 1.27)
+				)
+				(hide yes)
+			)
+		)
+		(pin "2"
+		)
+		(pin "1"
+		)
+		(instances
+			(project "DCDC_mid"
+				(path "/6223a5f4-c243-4547-8c88-bb7b5a32f283"
+					(reference "C10")
+					(unit 1)
+				)
+			)
+		)
+	)
+	(symbol
 		(lib_id "Mechanical:MountingHole_Pad")
 		(at 212.09 46.99 0)
@@
 					(unit 1)
 				)
+			)
+		)
+	)
+	(symbol
+		(lib_id "power:GND")
+		(at 95.25 146.05 0)
+		(unit 1)
+		(exclude_from_sim no)
+		(in_bom yes)
+		(on_board yes)
+		(dnp no)
+		(fields_autoplaced yes)
+		(property "Reference" "#PWR021"
+			(at 95.25 152.4 0)
+			(effects
+				(font
+					(size 1.27 1.27)
+				)
+				(hide yes)
+			)
+		)
+		(property "Value" "GND"
+			(at 95.25 150.1831 0)
+			(effects
+				(font
+					(size 1.27 1.27)
+				)
+			)
+		)
+		(property "Footprint" ""
+			(at 95.25 146.05 0)
+			(effects
+				(font
+					(size 1.27 1.27)
+				)
+				(hide yes)
+			)
+		)
+		(property "Datasheet" ""
+			(at 95.25 146.05 0)
+			(effects
+				(font
+					(size 1.27 1.27)
+				)
+				(hide yes)
+			)
+		)
+		(property "Description" ""
+			(at 95.25 146.05 0)
+			(effects
+				(font
+					(size 1.27 1.27)
+				)
+				(hide yes)
+			)
+		)
+		(pin "1"
+		)
+		(instances
+			(project "DCDC_mid"
+				(path "/6223a5f4-c243-4547-8c88-bb7b5a32f283"
+					(reference "#PWR021")
+					(unit 1)
+				)

Commit message: DCDCmid Andere Transistoren
Parts:
- removed Q1, Q2: BD139, Package_TO_SOT_THT:TO-126-3_Vertical, symbol Transistor_BJT:BD139
- removed Q3: BD140, Package_TO_SOT_THT:TO-126-3_Vertical, symbol Transistor_BJT:BD140
- added F1: Fuse, Fuse:Fuse_Littelfuse_372_D8.50mm, symbol Device:Fuse
- added Q1: FTZ953, Package_TO_SOT_SMD:SOT-223-3_TabPin2, symbol Transistor_BJT:BCP53
- added Q5, Q6: FTZ853, Package_TO_SOT_SMD:SOT-223-3_TabPin2, symbol Transistor_BJT:BCP56
Connections:
- net +VDC: now also F1.2, Q5.2 (C), Q5.4 (C); no longer D1.1 (K), D2.1 (K)
- net GND: now also Q1.2 (C), Q1.4 (C), Q6.3 (E)
- net at R6.2: now also Q1.1 (B), Q5.1 (B), Q6.2 (C), Q6.4 (C)
- net at R5.2, U2.7: now also Q6.1 (B)
- net at R7.1: now also Q1.3 (E), Q5.3 (E)
- new net: D1.1 (K), D2.1 (K), F1.1

Commit message: Powerstage2 und HBrücke3 Aufgebaut und verbesserungen eingearbeitet.
Parts:
- R6: value 100 -> 470
Other:
- note added: "R6 wird warm"
- note added: "z.B. IRF4905"
Changed lines of the file:
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@@
+		)
+	)
+	(text "R6 wird warm"
+		(exclude_from_sim no)
+		(at 92.71 39.37 0)
+		(effects
+			(font
+				(size 1.27 1.27)
+			)
 		)
 	)
@@
 			)
 			(justify left bottom)
+		)
+	)
+	(text "z.B. IRF4905"
+		(exclude_from_sim no)
+		(at 144.78 68.58 0)
+		(effects
+			(font
+				(size 1.27 1.27)
+			)
 		)
 	)
@@
 			)
 		)
-		(property "Value" "100"
+		(property "Value" "470"
 			(at 104.648 53.2821 0)
 			(effects
