File: OP-D-Amp/Addierer-Analog.kicad_sch (KiCad schematic)
At the start: 26 parts, among them J1 Conn_01x04_Pin, J2 Conn_01x04_Pin, U3 NE5532, U4 NE5532, U5 LMV393

Commit message: Kleinere Änderungen
Parts:
- added C21: 1u, Capacitor_THT:C_Axial_L3.8mm_D2.6mm_P7.50mm_Horizontal, symbol Device:C
- R8: value 10k -> 100k
Connections:
- net at TP5.2: now also C21.1; no longer R11.1
- new net: C21.2, R11.1
Other:
- moved on the sheet: R12
Changed lines of the file:
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@@
 	(paper "A4")
 	(title_block
-		(date "2023-12-21")
-		(rev "V2")
-		(comment 1 "Verbesserungen aus 1. Version eingearbeitet. ")
-		(comment 2 "Fehler falsche Footprints korrigiert, Schaltungsänderungen")
+		(date "2024-09-27")
+		(rev "V3")
+		(comment 1 "Verbesserungen aus 2. Version eingearbeitet. ")
 	)
 	(junction
@@
 	(wire
 		(pts
-			(xy 210.82 97.79) (xy 210.82 104.14)
+			(xy 119.38 99.06) (xy 132.08 99.06)
 		)
 		(stroke
@@
 	(wire
 		(pts
-			(xy 194.31 109.22) (xy 194.31 115.57)
+			(xy 210.82 97.79) (xy 210.82 104.14)
 		)
 		(stroke
@@
 	(wire
 		(pts
-			(xy 228.6 118.11) (xy 234.95 118.11)
+			(xy 194.31 109.22) (xy 194.31 115.57)
 		)
 		(stroke
@@
 	(wire
 		(pts
-			(xy 110.49 165.1) (xy 114.3 165.1)
+			(xy 228.6 118.11) (xy 234.95 118.11)
 		)
 		(stroke
@@
 	(wire
 		(pts
-			(xy 143.51 111.76) (xy 143.51 109.22)
+			(xy 110.49 165.1) (xy 114.3 165.1)
 		)
 		(stroke
@@
 	(wire
 		(pts
+			(xy 143.51 118.11) (xy 139.7 118.11)
+		)
+		(stroke
+			(width 0)
+			(type default)
+		)
+	)
+	(wire
+		(pts
 			(xy 91.44 158.75) (xy 91.44 163.83)
 		)
@@
 	(wire
 		(pts
+			(xy 143.51 109.22) (xy 143.51 118.11)
+		)
+		(stroke
+			(width 0)
+			(type default)
+		)
+	)
+	(wire
+		(pts
 			(xy 62.23 101.6) (xy 66.04 101.6)
 		)
@@
 	(wire
 		(pts
-			(xy 124.46 111.76) (xy 132.08 111.76)
+			(xy 124.46 118.11) (xy 132.08 118.11)
 		)
 		(stroke
@@
 	(wire
 		(pts
-			(xy 139.7 111.76) (xy 143.51 111.76)
-		)
-		(stroke
-			(width 0)
-			(type default)
-		)
-	)
-	(wire
-		(pts
 			(xy 62.23 110.49) (xy 62.23 101.6)
 		)
@@
 	(wire
 		(pts
-			(xy 102.87 99.06) (xy 132.08 99.06)
+			(xy 102.87 99.06) (xy 111.76 99.06)
 		)
 		(stroke
@@
 	(wire
 		(pts
-			(xy 124.46 156.21) (xy 124.46 111.76)
+			(xy 124.46 156.21) (xy 124.46 118.11)
 		)
 		(stroke
@@
 			)
 		)
-		(property "Value" "10k"
+		(property "Value" "100k"
 			(at 72.39 106.68 90)
 			(effects
@@
 	(symbol
 		(lib_id "Device:R")
-		(at 135.89 111.76 90)
+		(at 135.89 118.11 90)
 		(unit 1)
 		(exclude_from_sim no)
@@
 		(fields_autoplaced yes)
 		(property "Reference" "R12"
-			(at 135.89 106.5997 90)
+			(at 135.89 112.9497 90)
 			(effects
 				(font
@@
 		)
 		(property "Value" "10k"
-			(at 135.89 109.0239 90)
+			(at 135.89 115.3739 90)
 			(effects
 				(font
@@
 		)
 		(property "Footprint" "Resistor_SMD:R_0805_2012Metric_Pad1.20x1.40mm_HandSolder"
-			(at 135.89 113.538 90)
+			(at 135.89 119.888 90)
 			(effects
 				(font
@@
 		)
 		(property "Datasheet" "~"
-			(at 135.89 111.76 0)
+			(at 135.89 118.11 0)
 			(effects
 				(font
@@
 		)
 		(property "Description" ""
-			(at 135.89 111.76 0)
+			(at 135.89 118.11 0)
 			(effects
 				(font
@@
 					(unit 1)
 				)
+			)
+		)
+	)
+	(symbol
+		(lib_id "Device:C")
+		(at 115.57 99.06 90)
+		(unit 1)
+		(exclude_from_sim no)
+		(in_bom yes)
+		(on_board yes)
+		(dnp no)
+		(property "Reference" "C21"
+			(at 114.935 96.52 0)
+			(effects
+				(font
+					(size 1.27 1.27)
+				)
+				(justify left)
+			)
+		)
+		(property "Value" "1u"
+			(at 116.205 96.52 0)
+			(effects
+				(font
+					(size 1.27 1.27)
+				)
+				(justify left)
+			)
+		)
+		(property "Footprint" "Capacitor_THT:C_Axial_L3.8mm_D2.6mm_P7.50mm_Horizontal"
+			(at 119.38 98.0948 0)
+			(effects
+				(font
+					(size 1.27 1.27)
+				)
+				(hide yes)
+			)
+		)
+		(property "Datasheet" "~"
+			(at 115.57 99.06 0)
+			(effects
+				(font
+					(size 1.27 1.27)
+				)
+				(hide yes)
+			)
+		)
+		(property "Description" ""
+			(at 115.57 99.06 0)
+			(effects
+				(font
+					(size 1.27 1.27)
+				)
+				(hide yes)
+			)
+		)
+		(pin "1"
+		)
+		(pin "2"
+		)
+		(instances
+			(project "OP-D-Amp"
+				(path "/a2afb3b1-1b3e-46fd-a0bf-9e80fa6f6a60/e73c7bc6-f9a8-4517-8e4a-e472ea21b2cb"
+					(reference "C21")
+					(unit 1)
+				)

Commit message: Anlegen Projekt Useless Relais Addierer
Parts:
- added 150pf: C, symbol Device:C
Connections:
- net at R8.2, TP5.1, U4.7: now also 150pf.2
- net at R8.1, RV1.2, U4.6 (-): now also 150pf.1
- net OSC_inv: no longer names the net of J1.4 (Pin_4)
Other:
- note added: "43K"
- note added: "LM4562"
Changed lines of the file:
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@@
 	(paper "A4")
 	(title_block
-		(date "2024-09-27")
-		(rev "V3")
+		(date "2025-05-13")
+		(rev "V4")
 		(comment 1 "Verbesserungen aus 2. Version eingearbeitet. ")
+		(comment 2 "EIngang 150pF Rückkoplung engefügt, Verstärkung eingestellt")
+	)
+	(text "LM4562"
+		(exclude_from_sim no)
+		(at 100.33 142.24 0)
+		(effects
+			(font
+				(size 1.27 1.27)
+			)
+		)
+	)
+	(text "43K"
+		(exclude_from_sim no)
+		(at 106.68 170.18 0)
+		(effects
+			(font
+				(size 1.27 1.27)
+			)
+		)
+	)
+	(text "43K"
+		(exclude_from_sim no)
+		(at 76.2 114.3 0)
+		(effects
+			(font
+				(size 1.27 1.27)
+			)
+		)
 	)
 	(junction
@@
 	)
 	(junction
+		(at 81.28 110.49)
+		(diameter 0)
+		(color 0 0 0 0)
+	)
+	(junction
 		(at 184.15 96.52)
 		(diameter 0)
@@
 	(wire
 		(pts
+			(xy 62.23 125.73) (xy 67.31 125.73)
+		)
+		(stroke
+			(width 0)
+			(type default)
+		)
+	)
+	(wire
+		(pts
 			(xy 45.72 106.68) (xy 45.72 110.49)
 		)
@@
 	(wire
 		(pts
-			(xy 30.48 64.77) (xy 35.56 64.77)
-		)
-		(stroke
-			(width 0)
-			(type default)
-		)
-	)
-	(wire
-		(pts
 			(xy 81.28 99.06) (xy 92.71 99.06)
 		)
@@
 	(wire
 		(pts
+			(xy 74.93 125.73) (xy 81.28 125.73)
+		)
+		(stroke
+			(width 0)
+			(type default)
+		)
+	)
+	(wire
+		(pts
 			(xy 210.82 118.11) (xy 220.98 118.11)
 		)
@@
 	(wire
 		(pts
+			(xy 62.23 110.49) (xy 62.23 125.73)
+		)
+		(stroke
+			(width 0)
+			(type default)
+		)
+	)
+	(wire
+		(pts
 			(xy 62.23 110.49) (xy 68.58 110.49)
 		)
@@
 		(pts
 			(xy 30.48 59.69) (xy 50.8 59.69)
+		)
+		(stroke
+			(width 0)
+			(type default)
+		)
+	)
+	(wire
+		(pts
+			(xy 81.28 125.73) (xy 81.28 110.49)
 		)
 		(stroke
@@
 		)
 	)
-	(global_label "OSC_inv"
-		(shape input)
-		(at 35.56 64.77 0)
-		(effects
-			(font
-				(size 1.27 1.27)
-			)
-			(justify left)
-		)
-		(property "Intersheetrefs" "${INTERSHEET_REFS}"
-			(at 35.56 64.77 0)
-			(effects
-				(font
-					(size 1.27 1.27)
-				)
-				(hide yes)
-			)
-		)
-	)
 	(global_label "Sign_ein"
 		(shape input)
@@
 		)
 		(property "Value" "R_Potentiometer"
-			(at 73.914 117.856 0)
+			(at 58.42 104.14 0)
 			(effects
 				(font
@@
 					(unit 1)
 				)
+			)
+		)
+	)
+	(symbol
+		(lib_id "Device:C")
+		(at 71.12 125.73 90)
+		(unit 1)
+		(exclude_from_sim no)
+		(in_bom yes)
+		(on_board yes)
+		(dnp no)
+		(fields_autoplaced yes)
+		(property "Reference" "150pf"
+			(at 71.12 118.11 90)
+			(effects
+				(font
+					(size 1.27 1.27)
+				)
+			)
+		)
+		(property "Value" "C"
+			(at 71.12 120.65 90)
+			(effects
+				(font
+					(size 1.27 1.27)
+				)
+			)
+		)
+		(property "Footprint" ""
+			(at 74.93 124.7648 0)
+			(effects
+				(font
+					(size 1.27 1.27)
+				)
+				(hide yes)
+			)
+		)
+		(property "Datasheet" "~"
+			(at 71.12 125.73 0)
+			(effects
+				(font
+					(size 1.27 1.27)
+				)
+				(hide yes)
+			)
+		)
+		(property "Description" "Unpolarized capacitor"
+			(at 71.12 125.73 0)
+			(effects
+				(font
+					(size 1.27 1.27)
+				)
+				(hide yes)
+			)
+		)
+		(pin "2"
+		)
+		(pin "1"
+		)
+		(instances
+			(project ""
+				(path "/a2afb3b1-1b3e-46fd-a0bf-9e80fa6f6a60/e73c7bc6-f9a8-4517-8e4a-e472ea21b2cb"
+					(reference "150pf")
+					(unit 1)
+				)
