File: OP-D-Amp/Netzteil.kicad_sch (KiCad schematic)
At the start: 19 parts, among them J3 Conn_01x04_Pin, U1 40106, U2 4027, U3 NE5532, U4 NE5532, U5 LMV393

Commit message: Kleinere Änderungen
Changed lines of the file:
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@@
+	)
+	(junction
+		(at 55.245 75.565)
+		(diameter 0)
+		(color 0 0 0 0)
 	)
 	(junction
@@
 	)
 	(junction
-		(at 55.245 75.565)
-		(diameter 0)
-		(color 0 0 0 0)
-	)
-	(junction
 		(at 151.13 146.685)
 		(diameter 0)
@@
 	(wire
 		(pts
+			(xy 55.88 75.565) (xy 55.88 72.39)
+		)
+		(stroke
+			(width 0)
+			(type default)
+		)
+	)
+	(wire
+		(pts
 			(xy 125.095 146.685) (xy 115.57 146.685)
 		)
@@
 	(wire
 		(pts
-			(xy 55.245 75.565) (xy 55.245 74.295)
-		)
-		(stroke
-			(width 0)
-			(type default)
-		)
-	)
-	(wire
-		(pts
 			(xy 46.355 32.385) (xy 46.355 33.655)
 		)
@@
 	(wire
 		(pts
+			(xy 55.245 106.68) (xy 55.245 100.965)
+		)
+		(stroke
+			(width 0)
+			(type default)
+		)
+	)
+	(wire
+		(pts
 			(xy 72.39 99.06) (xy 72.39 96.52)
 		)
@@
 	(wire
 		(pts
+			(xy 55.245 75.565) (xy 55.88 75.565)
+		)
+		(stroke
+			(width 0)
+			(type default)
+		)
+	)
+	(wire
+		(pts
 			(xy 42.545 85.725) (xy 42.545 75.565)
 		)
@@
 	(wire
 		(pts
-			(xy 55.245 106.045) (xy 55.245 100.965)
-		)
-		(stroke
-			(width 0)
-			(type default)
-		)
-	)
-	(wire
-		(pts
 			(xy 151.13 140.97) (xy 151.13 146.685)
 		)
@@
 		(pts
 			(xy 177.165 142.875) (xy 177.165 144.78)
+		)
+		(stroke
+			(width 0)
+			(type default)
+		)
+	)
+	(wire
+		(pts
+			(xy 55.88 106.68) (xy 55.245 106.68)
 		)
 		(stroke
@@
 	(symbol
 		(lib_id "power:+12V")
-		(at 55.245 74.295 0)
+		(at 55.88 72.39 0)
 		(unit 1)
 		(exclude_from_sim no)
@@
 		(dnp no)
 		(property "Reference" "#PWR04"
-			(at 55.245 78.105 0)
+			(at 55.88 76.2 0)
 			(effects
 				(font
@@
 		)
 		(property "Value" "+12V"
-			(at 55.626 69.9008 0)
+			(at 56.261 67.9958 0)
 			(effects
 				(font
@@
 		)
 		(property "Footprint" ""
-			(at 55.245 74.295 0)
+			(at 55.88 72.39 0)
 			(effects
 				(font
@@
 		)
 		(property "Datasheet" ""
-			(at 55.245 74.295 0)
-			(effects
-				(font
-					(size 1.27 1.27)
-				)
-				(hide yes)
-			)
-		)
-		(property "Description" ""
-			(at 55.245 74.295 0)
+			(at 55.88 72.39 0)
+			(effects
+				(font
+					(size 1.27 1.27)
+				)
+				(hide yes)
+			)
+		)
+		(property "Description" ""
+			(at 55.88 72.39 0)
 			(effects
 				(font
@@
 	(symbol
 		(lib_id "power:GND")
-		(at 55.245 106.045 0)
+		(at 55.88 106.68 0)
 		(unit 1)
 		(exclude_from_sim no)
@@
 		(dnp no)
 		(property "Reference" "#PWR05"
-			(at 55.245 112.395 0)
+			(at 55.88 113.03 0)
 			(effects
 				(font
@@
 		)
 		(property "Value" "GND"
-			(at 55.372 110.4392 0)
+			(at 56.007 111.0742 0)
 			(effects
 				(font
@@
 		)
 		(property "Footprint" ""
-			(at 55.245 106.045 0)
+			(at 55.88 106.68 0)
 			(effects
 				(font
@@
 		)
 		(property "Datasheet" ""
-			(at 55.245 106.045 0)
-			(effects
-				(font
-					(size 1.27 1.27)
-				)
-				(hide yes)
-			)
-		)
-		(property "Description" ""
-			(at 55.245 106.045 0)
-			(effects
-				(font
+			(at 55.88 106.68 0)
+			(effects
+				(font
+					(size 1.27 1.27)
+				)
+				(hide yes)
+			)
+		)
+		(property "Description" ""
+			(at 55.88 106.68 0)
+			(effects
+				(font

Commit message: Anlegen Projekt Useless Relais Addierer
Parts:
- renumbered C3 to C10, D1 to D3, D2 to D4
Changed lines of the file:
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@@
 (kicad_sch
-	(version 20231120)
+	(version 20250114)
 	(generator "eeschema")
-	(generator_version "8.0")
+	(generator_version "9.0")
 	(paper "A4")
 	(junction
@@
 		(on_board yes)
 		(dnp no)
-		(property "Reference" "#PWR04"
+		(property "Reference" "#PWR028"
 			(at 53.34 33.655 0)
 			(effects
@@
 		(on_board yes)
 		(dnp no)
-		(property "Reference" "#PWR03"
+		(property "Reference" "#PWR026"
 			(at 42.545 102.235 0)
 			(effects
@@
 		(on_board yes)
 		(dnp no)
-		(property "Reference" "C3"
+		(property "Reference" "C10"
 			(at 39.624 88.3666 0)
 			(effects
@@
 		(on_board yes)
 		(dnp no)
-		(property "Reference" "#PWR04"
+		(property "Reference" "#PWR030"
 			(at 55.88 76.2 0)
 			(effects
@@
 		(on_board yes)
 		(dnp no)
-		(property "Reference" "#PWR05"
+		(property "Reference" "#PWR031"
 			(at 55.88 113.03 0)
 			(effects
@@
 		(on_board yes)
 		(dnp no)
-		(property "Reference" "D2"
+		(property "Reference" "D4"
 			(at 44.45 24.3586 0)
 			(effects
@@
 		(on_board yes)
 		(dnp no)
-		(property "Reference" "D1"
+		(property "Reference" "D3"
 			(at 43.18 42.9514 0)
 			(effects
