File: OP-D-Amp/OP-D-Amp.kicad_pcb (KiCad board)
At the start: 2 copper layers, 73.7 x 72.4 mm, 60 parts, among them J1 Conn_01x04_Pin, J2 Conn_01x04_Pin, J3 Conn_01x04_Pin, SW1 SW_Wuerth_450301014042, U1 40106, U2 4027, U3 NE5532, U4 NE5532, U5 LMV393

Commit message: Kleinere Änderungen
Parts:
- removed the C5 at (182.9, 101.6)
- removed the TP3 at (162.5, 77.1)
- added C21: 1u, Capacitor_THT:C_Axial_L3.8mm_D2.6mm_P7.50mm_Horizontal, F.Cu at (159.2, 102.5)
- added R18: 1M, Resistor_SMD:R_0805_2012Metric_Pad1.20x1.40mm_HandSolder, F.Cu at (182.2, 87.0)
- R8: value 10k -> 100k
Connections:
- R11 pad 1: Net-(R11-Pad1) -> Net-(C21-Pad2)
- TP5 pad 2: Net-(R11-Pad1) -> Net-(C21-Pad1)
- U1 pad 10: Net-(TP1-Pad1) -> unconnected-(U1-Pad10)
- U1 pad 11: Osc -> +12V
- U1 pad 12: (no net) -> unconnected-(U1-Pad12)
- U1 pad 13: (no net) -> +12V
- U2 pad 14: Osc -> unconnected-(U2B-~{Q}-Pad14)
Routing:
- net +12V: track 294.5 -> 321.3 mm
- net Osc: track 25.5 -> 0.00 mm
- net OSC_inv: track 14.3 -> 0.00 mm
- net Net-(R11-Pad1): track 3.92 -> 0.00 mm
- net (no net): track 0.00 -> 3.92 mm

Commit message: Anlegen Projekt Useless Relais Addierer
Parts:
- moved TP1 3.15 mm to (153.1, 105.5)
- turned R18 to -90 degrees
Routing:
- net +12V: track 321.3 -> 301.8 mm
- net Net-(C21-Pad1): track 0.00 -> 6.18 mm
- net Net-(C21-Pad2): track 0.00 -> 5.77 mm
- net -12V: track 118.7 -> 124.2 mm
- net Net-(TP1-Pad1): track 12.6 -> 7.63 mm
- net Net-(SW1-C): track 37.8 -> 42.6 mm, vias 1 -> 2
- net (no net): track 3.92 -> 0.00 mm
- net Net-(C6-Pad2): track 14.6 -> 18.4 mm
- net GND: vias 39 -> 41
