File: OP-D-Amp/osziollator.kicad_sch (KiCad schematic)
At the start: 19 parts, among them SW1 SW_Wuerth_450301014042, U1 40106, U2 4027, U3 NE5532

Commit message: Version 2 für Herstellung
Parts:
- added unit 6 of U1
Connections:
- net +12V: now also U1.13
- no-connect marks 6 -> 7
Changed lines of the file:
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@@
+	)
+	(no_connect
+		(at 45.72 109.22)
 	)
 	(no_connect
@@
 	)
 	(symbol
+		(lib_id "4xxx:40106")
+		(at 38.1 109.22 0)
+		(unit 6)
+		(exclude_from_sim no)
+		(in_bom yes)
+		(on_board yes)
+		(dnp no)
+		(property "Reference" "U1"
+			(at 38.1 101.1682 0)
+			(effects
+				(font
+					(size 1.27 1.27)
+				)
+			)
+		)
+		(property "Value" "40106"
+			(at 38.1 103.4796 0)
+			(effects
+				(font
+					(size 1.27 1.27)
+				)
+			)
+		)
+		(property "Footprint" "Package_SO:SO-14_3.9x8.65mm_P1.27mm"
+			(at 38.1 109.22 0)
+			(effects
+				(font
+					(size 1.27 1.27)
+				)
+				(hide yes)
+			)
+		)
+		(property "Datasheet" "https://assets.nexperia.com/documents/data-sheet/HEF40106B.pdf"
+			(at 38.1 109.22 0)
+			(effects
+				(font
+					(size 1.27 1.27)
+				)
+				(hide yes)
+			)
+		)
+		(property "Description" ""
+			(at 38.1 109.22 0)
+			(effects
+				(font
+					(size 1.27 1.27)
+				)
+				(hide yes)
+			)
+		)
+		(pin "1"
+		)
+		(pin "2"
+		)
+		(pin "3"
+		)
+		(pin "4"
+		)
+		(pin "5"
+		)
+		(pin "6"
+		)
+		(pin "8"
+		)
+		(pin "9"
+		)
+		(pin "10"
+		)
+		(pin "11"
+		)
+		(pin "12"
+		)
+		(pin "13"
+		)
+		(pin "14"
+		)
+		(pin "7"
+		)
+		(instances
+			(project "OP-D-Amp"
+				(path "/a2afb3b1-1b3e-46fd-a0bf-9e80fa6f6a60/e48f986c-9b3e-49a4-ad94-2e09f65c8312"
+					(reference "U1")
+					(unit 6)
+				)
+			)
+		)
+	)
+	(symbol
 		(lib_id "Device:C")
 		(at 45.72 144.145 0)
@@
 				)
 			)
+		)
+	)
+	(symbol
+		(lib_id "power:+12V")
+		(at 30.48 109.22 0)
+		(unit 1)
+		(exclude_from_sim no)
+		(in_bom yes)
+		(on_board yes)
+		(dnp no)
+		(fields_autoplaced yes)
+		(property "Reference" "#PWR044"
+			(at 30.48 113.03 0)
+			(effects
+				(font
+					(size 1.27 1.27)
+				)
+				(hide yes)
+			)
+		)
+		(property "Value" "+12V"
+			(at 30.48 104.14 0)
+			(effects
+				(font
+					(size 1.27 1.27)
+				)
+			)
+		)
+		(property "Footprint" ""
+			(at 30.48 109.22 0)
+			(effects
+				(font
+					(size 1.27 1.27)
+				)
+				(hide yes)
+			)
+		)
+		(property "Datasheet" ""
+			(at 30.48 109.22 0)
+			(effects
+				(font
+					(size 1.27 1.27)
+				)
+				(hide yes)
+			)
+		)
+		(property "Description" ""
+			(at 30.48 109.22 0)
+			(effects
+				(font
+					(size 1.27 1.27)
+				)
+				(hide yes)
+			)
+		)
+		(pin "1"
+		)
+		(instances
+			(project "OP-D-Amp"
+				(path "/a2afb3b1-1b3e-46fd-a0bf-9e80fa6f6a60/e48f986c-9b3e-49a4-ad94-2e09f65c8312"
+					(reference "#PWR044")
+					(unit 1)
+				)
+			)

Commit message: Kleinere Änderungen
Parts:
- added R18: 1M, Resistor_SMD:R_0805_2012Metric_Pad1.20x1.40mm_HandSolder, symbol Device:R
Connections:
- net +12V: now also U1.11
- net at C6.1, R5.1, SW1.2 (C)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: now also R18.1
- net at TP1.1, U1.8: no longer U1.10
- net at C6.2, C7.1, U3.1: now also R18.2
- net Osc: no longer names the net of U2.14 (~{Q})
- net Osc: no longer U1.11
- no-connect marks 7 -> 9
Other:
- moved on the sheet: R5, U1E
Changed lines of the file:
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@@
 	)
 	(junction
-		(at 152.4 88.9)
+		(at 191.77 106.68)
 		(diameter 0)
 		(color 0 0 0 0)
 	)
 	(junction
-		(at 88.9 139.7)
+		(at 152.4 88.9)
 		(diameter 0)
 		(color 0 0 0 0)
 	)
 	(junction
-		(at 142.24 88.9)
+		(at 88.9 139.7)
 		(diameter 0)
 		(color 0 0 0 0)
 	)
 	(junction
-		(at 132.08 156.21)
+		(at 142.24 88.9)
 		(diameter 0)
 		(color 0 0 0 0)
 	)
 	(junction
-		(at 153.67 137.16)
+		(at 137.16 88.9)
 		(diameter 0)
 		(color 0 0 0 0)
 	)
 	(junction
-		(at 137.16 88.9)
+		(at 207.01 99.06)
 		(diameter 0)
 		(color 0 0 0 0)
@@
 	)
 	(no_connect
+		(at 132.08 142.24)
+	)
+	(no_connect
 		(at 46.99 72.39)
 	)
@@
 	)
 	(no_connect
+		(at 76.2 106.68)
+	)
+	(no_connect
 		(at 45.72 109.22)
 	)
@@
 	(wire
 		(pts
-			(xy 132.08 142.24) (xy 132.08 156.21)
-		)
-		(stroke
-			(width 0)
-			(type default)
-		)
-	)
-	(wire
-		(pts
 			(xy 142.24 101.6) (xy 142.24 105.41)
 		)
@@
 	(wire
 		(pts
-			(xy 152.4 156.21) (xy 153.67 156.21)
+			(xy 199.39 106.68) (xy 207.01 106.68)
 		)
 		(stroke
@@
 	(wire
 		(pts
-			(xy 132.08 156.21) (xy 132.08 161.29)
+			(xy 45.72 140.335) (xy 45.72 139.7)
 		)
 		(stroke
@@
 	(wire
 		(pts
-			(xy 132.08 156.21) (xy 137.16 156.21)
+			(xy 123.19 88.9) (xy 129.54 88.9)
 		)
 		(stroke
@@
 	(wire
 		(pts
-			(xy 45.72 140.335) (xy 45.72 139.7)
+			(xy 107.95 139.7) (xy 116.84 139.7)
 		)
 		(stroke
@@
 	(wire
 		(pts
-			(xy 123.19 88.9) (xy 129.54 88.9)
+			(xy 60.96 134.62) (xy 62.23 134.62)
 		)
 		(stroke
@@
 	(wire
 		(pts
-			(xy 107.95 139.7) (xy 116.84 139.7)
+			(xy 88.9 119.38) (xy 57.15 119.38)
 		)
 		(stroke
@@
 	(wire
 		(pts
-			(xy 60.96 134.62) (xy 62.23 134.62)
+			(xy 191.77 99.06) (xy 191.77 106.68)
 		)
 		(stroke
@@
 	(wire
 		(pts
-			(xy 153.67 137.16) (xy 153.67 156.21)
+			(xy 137.16 88.9) (xy 142.24 88.9)
 		)
 		(stroke
@@
 	(wire
 		(pts
-			(xy 88.9 119.38) (xy 57.15 119.38)
+			(xy 132.08 137.16) (xy 137.16 137.16)
 		)
 		(stroke
@@
 	(wire
 		(pts
-			(xy 137.16 88.9) (xy 142.24 88.9)
+			(xy 88.9 139.7) (xy 92.71 139.7)
 		)
 		(stroke
@@
 	(wire
 		(pts
-			(xy 132.08 137.16) (xy 137.16 137.16)
+			(xy 223.52 91.44) (xy 232.41 91.44)
 		)
 		(stroke
@@
 	(wire
 		(pts
-			(xy 88.9 139.7) (xy 92.71 139.7)
+			(xy 168.91 140.97) (xy 175.26 140.97)
 		)
 		(stroke
@@
 	(wire
 		(pts
-			(xy 223.52 91.44) (xy 232.41 91.44)
+			(xy 45.72 139.7) (xy 57.15 139.7)
 		)
 		(stroke
@@
 	(wire
 		(pts
-			(xy 168.91 140.97) (xy 175.26 140.97)
+			(xy 113.03 142.24) (xy 116.84 142.24)
 		)
 		(stroke
@@
 	(wire
 		(pts
-			(xy 45.72 139.7) (xy 57.15 139.7)
+			(xy 207.01 106.68) (xy 207.01 99.06)
 		)
 		(stroke
@@
 	(wire
 		(pts
-			(xy 113.03 142.24) (xy 116.84 142.24)
+			(xy 137.16 88.9) (xy 137.16 93.98)
 		)
 		(stroke
@@
 	(wire
 		(pts
-			(xy 137.16 88.9) (xy 137.16 93.98)
+			(xy 60.96 104.14) (xy 60.96 106.68)
 		)
 		(stroke
@@
 	(wire
 		(pts
-			(xy 152.4 137.16) (xy 153.67 137.16)
+			(xy 152.4 137.16) (xy 158.75 137.16)
 		)
 		(stroke
@@
 	(wire
 		(pts
-			(xy 191.77 106.68) (xy 191.77 140.97)
+			(xy 191.77 106.68) (xy 191.77 120.65)
 		)
 		(stroke
@@
 	(wire
 		(pts
-			(xy 153.67 137.16) (xy 158.75 137.16)
+			(xy 177.8 99.06) (xy 177.8 91.44)
 		)
 		(stroke
@@
 	(wire
 		(pts
-			(xy 177.8 99.06) (xy 177.8 91.44)
+			(xy 191.77 128.27) (xy 191.77 140.97)
 		)
 		(stroke
@@
 		)
 	)
-	(global_label "Osc"
-		(shape input)
-		(at 132.08 161.29 0)
-		(effects
-			(font
-				(size 1.27 1.27)
-			)
-			(justify left)
-		)
-		(property "Intersheetrefs" "${INTERSHEET_REFS}"
-			(at 132.08 161.29 0)
-			(effects
-				(font
-					(size 1.27 1.27)
-				)
-				(hide yes)
-			)
-		)
-	)
 	(global_label "TRI"
 		(shape input)
@@
 		(on_board yes)
 		(dnp no)
-		(fields_autoplaced yes)
 		(property "Reference" "SW1"
 			(at 172.72 80.01 0)
@@
 		)
 		(property "Value" "SW_Wuerth_450301014042"
-			(at 172.72 82.55 0)
+			(at 177.8 64.77 0)
 			(effects
 				(font
@@
 	(symbol
 		(lib_id "4xxx:40106")
-		(at 144.78 156.21 0)
+		(at 68.58 106.68 0)
 		(unit 5)
 		(exclude_from_sim no)
@@
 		(dnp no)
 		(property "Reference" "U1"
-			(at 146.05 161.29 0)
+			(at 69.85 111.76 0)
 			(effects
 				(font
@@
 		)
 		(property "Value" "40106"
-			(at 144.78 150.4696 0)
+			(at 68.58 100.9396 0)
 			(effects
 				(font
@@
 		)
 		(property "Footprint" "Package_SO:SO-14_3.9x8.65mm_P1.27mm"
-			(at 144.78 156.21 0)
+			(at 68.58 106.68 0)
 			(effects
 				(font
@@
 		)
 		(property "Datasheet" "https://assets.nexperia.com/documents/data-sheet/HEF40106B.pdf"
-			(at 144.78 156.21 0)
+			(at 68.58 106.68 0)
 			(effects
 				(font
@@
 		)
 		(property "Description" ""
-			(at 144.78 156.21 0)
+			(at 68.58 106.68 0)
 			(effects
 				(font
@@
 	)
 	(symbol
+		(lib_id "Device:R")
+		(at 195.58 106.68 90)
+		(unit 1)
+		(exclude_from_sim no)
+		(in_bom yes)
+		(on_board yes)
+		(dnp no)
+		(fields_autoplaced yes)
+		(property "Reference" "R18"
+			(at 195.58 100.33 90)
+			(effects
+				(font
+					(size 1.27 1.27)
+				)
+			)
+		)
+		(property "Value" "1M"
+			(at 195.58 102.87 90)
+			(effects
+				(font
+					(size 1.27 1.27)
+				)
+			)
+		)
+		(property "Footprint" "Resistor_SMD:R_0805_2012Metric_Pad1.20x1.40mm_HandSolder"
+			(at 195.58 108.458 90)
+			(effects
+				(font
+					(size 1.27 1.27)
+				)
+				(hide yes)
+			)
+		)
+		(property "Datasheet" "~"
+			(at 195.58 106.68 0)
+			(effects
+				(font
+					(size 1.27 1.27)
+				)
+				(hide yes)
+			)
+		)
+		(property "Description" ""
+			(at 195.58 106.68 0)
+			(effects
+				(font
+					(size 1.27 1.27)
+				)
+				(hide yes)
+			)
+		)
+		(pin "1"
+		)
+		(pin "2"
+		)
+		(instances
+			(project "OP-D-Amp"
+				(path "/a2afb3b1-1b3e-46fd-a0bf-9e80fa6f6a60/e48f986c-9b3e-49a4-ad94-2e09f65c8312"
+					(reference "R18")
+					(unit 1)
+				)
+			)
+		)
+	)
+	(symbol
 		(lib_id "Amplifier_Operational:NE5532")
 		(at 199.39 91.44 0)
@@
 	(symbol
 		(lib_id "Device:R")
-		(at 191.77 102.87 0)
+		(at 191.77 124.46 0)
 		(unit 1)
 		(exclude_from_sim no)
@@
 		(fields_autoplaced yes)
 		(property "Reference" "R5"
-			(at 193.548 101.6579 0)
+			(at 193.548 123.2479 0)
 			(effects
 				(font
@@
 		)
 		(property "Value" "75k"
-			(at 193.548 104.0821 0)
+			(at 193.548 125.6721 0)
 			(effects
 				(font
@@
 		)
 		(property "Footprint" "Resistor_SMD:R_0805_2012Metric_Pad1.20x1.40mm_HandSolder"
-			(at 189.992 102.87 90)
+			(at 189.992 124.46 90)
 			(effects
 				(font
@@
 		)
 		(property "Datasheet" "~"
-			(at 191.77 102.87 0)
+			(at 191.77 124.46 0)
 			(effects
 				(font
@@
 		)
 		(property "Description" ""
-			(at 191.77 102.87 0)
+			(at 191.77 124.46 0)
 			(effects
 				(font
@@
 					(unit 1)
 				)
+			)
+		)
+	)
+	(symbol
+		(lib_id "power:+12V")
+		(at 60.96 104.14 0)
+		(unit 1)
+		(exclude_from_sim no)
+		(in_bom yes)
+		(on_board yes)
+		(dnp no)
+		(property "Reference" "#PWR045"
+			(at 60.96 107.95 0)
+			(effects
+				(font
+					(size 1.27 1.27)
+				)
+				(hide yes)
+			)
+		)
+		(property "Value" "+12V"
+			(at 60.96 100.33 0)
+			(effects
+				(font
+					(size 1.27 1.27)
+				)
+			)
+		)
+		(property "Footprint" ""
+			(at 60.96 104.14 0)
+			(effects
+				(font
+					(size 1.27 1.27)
+				)
+				(hide yes)
+			)
+		)
+		(property "Datasheet" ""
+			(at 60.96 104.14 0)
+			(effects
+				(font
+					(size 1.27 1.27)
+				)
+				(hide yes)
+			)
+		)
+		(property "Description" ""
+			(at 60.96 104.14 0)
+			(effects
+				(font
+					(size 1.27 1.27)
+				)
+				(hide yes)
+			)
+		)
+		(pin "1"
+		)
+		(instances
+			(project "OP-D-Amp"
+				(path "/a2afb3b1-1b3e-46fd-a0bf-9e80fa6f6a60/e48f986c-9b3e-49a4-ad94-2e09f65c8312"
+					(reference "#PWR045")
+					(unit 1)
+				)
