File: Breadboard/PB_OP-V2/PB_OP-V2.kicad_sch (KiCad schematic)
At the start: 24 parts, among them J1 Conn_01x02_Pin, J2 Conn_01x02_Pin, J3 Conn_01x08_Pin, U1 NE5532

Commit message: Useless Adder auf V2.0 gebracht. Software finalisiert, Platine benötigt noch Arbeit
Other:
- moved on the sheet: R1
Changed lines of the file:
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@@
+	(wire
+		(pts
+			(xy 160.02 55.88) (xy 163.83 55.88)
+		)
+		(stroke
+			(width 0)
+			(type default)
+		)
+	)
 	(wire
 		(pts
@@
 	(wire
 		(pts
-			(xy 132.08 57.15) (xy 165.1 57.15)
+			(xy 132.08 55.88) (xy 152.4 55.88)
 		)
 		(stroke
@@
 	(wire
 		(pts
-			(xy 132.08 87.63) (xy 132.08 57.15)
+			(xy 132.08 87.63) (xy 132.08 55.88)
 		)
 		(stroke
@@
 	(wire
 		(pts
+			(xy 163.83 55.88) (xy 163.83 57.15)
+		)
+		(stroke
+			(width 0)
+			(type default)
+		)
+	)
+	(wire
+		(pts
 			(xy 36.83 133.35) (xy 41.91 133.35)
 		)
@@
 		(pts
 			(xy 193.04 90.17) (xy 198.12 90.17)
+		)
+		(stroke
+			(width 0)
+			(type default)
+		)
+	)
+	(wire
+		(pts
+			(xy 163.83 57.15) (xy 172.72 57.15)
 		)
 		(stroke
@@
 	(symbol
 		(lib_id "Device:R")
-		(at 168.91 57.15 90)
+		(at 156.21 55.88 90)
 		(unit 1)
 		(exclude_from_sim no)
@@
 		(dnp no)
 		(property "Reference" "R1"
-			(at 168.91 57.15 90)
+			(at 156.21 55.88 90)
 			(effects
 				(font
@@
 		)
 		(property "Value" "R"
-			(at 168.91 54.4139 90)
+			(at 156.21 53.1439 90)
 			(effects
 				(font
@@
 		)
 		(property "Footprint" "Resistor_THT:R_Axial_DIN0204_L3.6mm_D1.6mm_P7.62mm_Horizontal"
-			(at 168.91 58.928 90)
+			(at 156.21 57.658 90)
 			(effects
 				(font
@@
 		)
 		(property "Datasheet" "~"
-			(at 168.91 57.15 0)
+			(at 156.21 55.88 0)
 			(effects
 				(font
@@
 		)
 		(property "Description" ""
-			(at 168.91 57.15 0)
-			(effects
-				(font
+			(at 156.21 55.88 0)
+			(effects
+				(font
