File: Useless Relais Addierer/RelaisAddierer/RelaisAddierer.kicad_sch (KiCad schematic)
At the start: 254 parts, among them J1 Conn_01x08_Pin, J2 Barrel_Jack, K201 HK19F-DCxxV-SHC, K202 HK19F-DCxxV-SHC, K203 HK19F-DCxxV-SHC, K204 HK19F-DCxxV-SHC, K205 HK19F-DCxxV-SHC, K206 HK19F-DCxxV-SHC, K207 HK19F-DCxxV-SHC, K208 HK19F-DCxxV-SHC, K209 HK19F-DCxxV-SHC, K210 HK19F-DCxxV-SHC, K211 HK19F-DCxxV-SHC, K212 HK19F-DCxxV-SHC, K213 HK19F-DCxxV-SHC, K214 HK19F-DCxxV-SHC, K215 HK19F-DCxxV-SHC, K216 HK19F-DCxxV-SHC, K217 HK19F-DCxxV-SHC, K218 HK19F-DCxxV-SHC, K219 HK19F-DCxxV-SHC, K220 HK19F-DCxxV-SHC, K221 HK19F-DCxxV-SHC, K222 HK19F-DCxxV-SHC, K223 HK19F-DCxxV-SHC, K224 HK19F-DCxxV-SHC, K225 HK19F-DCxxV-SHC, K226 HK19F-DCxxV-SHC, K227 HK19F-DCxxV-SHC, K228 HK19F-DCxxV-SHC, K229 HK19F-DCxxV-SHC, K230 HK19F-DCxxV-SHC, K231 HK19F-DCxxV-SHC, K232 HK19F-DCxxV-SHC, Q1 BC847, Q10 BC847, Q11 DMP3099L, Q12 DMP3099L, Q13 DMP3099L, Q14 DMP3099L, Q15 DMP3099L, Q16 DMP3099L, Q17 BC847, Q18 BC847, Q19 BC847, Q2 BC847, Q20 BC847, Q201 BSS138, Q202 BSS138, Q21 BC847, Q22 DMP3099L, Q23 BC847, Q24 BC847, Q25 DMP3099L, Q26 BC847, Q27 DMP3099L, Q28 DMP3099L, Q29 DMP3099L, Q3 BC847, Q30 DMP3099L, Q31 DMP3099L, Q32 DMP3099L, Q4 BC847, Q5 BC847, Q6 DMP3099L, Q7 BC847, Q8 BC847, Q9 DMP3099L, SW1 RotaryEncoder_Switch, SW2 RotaryEncoder_Switch, U1 TCA9534, U2 TCA9534, U3 TCA9534, U4 uA7805

Commit message: Useless Adder auf V2.0 gebracht. Software finalisiert, Platine benötigt noch Arbeit
Parts:
- D2, D201, D202, D203, D204, D205, D206, D207, D208, D209, D210, D211, D212, D213, D214, D215, D216, D217, D218, D219, D220, D221, D222, D223, D224, D225, D226, D227, D228, D229, D230, D231, D232: footprint Diode_SMD:D_SOD-523 -> Diode_SMD:D_SMF
- D51, D52, D53, D54, D55, D56, D57, D58: footprint Diode_SMD:D_SMF -> Diode_SMD:D_MiniMELF
- Q6: value DMP3099L -> PJM10H01PSA
Connections:
- net +12V: now also K201.11, K202.11, K210.11; no longer K201.21
- net at K207.12, K208.14: now also K216.22
- net Carry_Bit6_neg: now reaches K222.11, K230.11
- net Carry_Bit6_neg: now also K228.21
- net Carry_Bit7_neg: now reaches K230.21
- net Carry_Bit7_neg: now also K224.11, K232.11
- net at K230.22: now also K221.12, K222.14
- net at K230.24: now also K222.12
- net at K202.12: now also K210.24
- net at K201.12, K202.14: now also K210.22
- net Carry_Bit3_neg: now reaches K208.11, K216.11
- net Carry_Bit3_neg: now also K214.21
- net at K208.12: now also K216.24
- net Carry_Bit5_neg: now reaches K220.11, K228.11
- net Carry_Bit5_neg: now also K226.21
- net at K228.22: now also K219.12, K220.14
- net at K228.24: now also K220.12
- net Carry_Bit1_neg: now reaches K204.11, K212.11
- net Carry_Bit1_neg: now also K210.21
- net Carry_Bit2_neg: now reaches K212.21
- net Carry_Bit2_neg: now also K206.11, K214.11
- net at K212.22: now also K203.12, K204.14
- net at K212.24: now also K204.12
- net Carry_Bit4_neg: now reaches K216.21
- net Carry_Bit4_neg: now also K218.11, K226.11
- net at K226.22: now also K217.12, K218.14
- net at K226.24: now also K218.12
Other:
- note added: "Ausgang Byte A"
- note added: "Ausgang Byte B"
- note added: "Display"
- note added: "Eingang Ergebnis Bit"
- note added: "Netzteil"
- note added: "SSD11306 i2c"
- moved on the sheet: D34, D35, D36, D37, D38, D39, D40, D41, H2, H3, H4, H5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
