File: Useless Relais Addierer/RelaisAddierer/RelaisAddierer.kicad_pcb (KiCad board)
At the start: 2 copper layers, 290.1 x 175 mm, 254 parts, among them J1 Conn_01x08_Pin, J2 Barrel_Jack, K201 HK19F-DCxxV-SHC, K202 HK19F-DCxxV-SHC, K203 HK19F-DCxxV-SHC, K204 HK19F-DCxxV-SHC, K205 HK19F-DCxxV-SHC, K206 HK19F-DCxxV-SHC, K207 HK19F-DCxxV-SHC, K208 HK19F-DCxxV-SHC, K209 HK19F-DCxxV-SHC, K210 HK19F-DCxxV-SHC, K211 HK19F-DCxxV-SHC, K212 HK19F-DCxxV-SHC, K213 HK19F-DCxxV-SHC, K214 HK19F-DCxxV-SHC, K215 HK19F-DCxxV-SHC, K216 HK19F-DCxxV-SHC, K217 HK19F-DCxxV-SHC, K218 HK19F-DCxxV-SHC, K219 HK19F-DCxxV-SHC, K220 HK19F-DCxxV-SHC, K221 HK19F-DCxxV-SHC, K222 HK19F-DCxxV-SHC, K223 HK19F-DCxxV-SHC, K224 HK19F-DCxxV-SHC, K225 HK19F-DCxxV-SHC, K226 HK19F-DCxxV-SHC, K227 HK19F-DCxxV-SHC, K228 HK19F-DCxxV-SHC, K229 HK19F-DCxxV-SHC, K230 HK19F-DCxxV-SHC, K231 HK19F-DCxxV-SHC, K232 HK19F-DCxxV-SHC, Q1 BC847, Q10 BC847, Q11 DMP3099L, Q12 DMP3099L, Q13 DMP3099L, Q14 DMP3099L, Q15 DMP3099L, Q16 DMP3099L, Q17 BC847, Q18 BC847, Q19 BC847, Q2 BC847, Q20 BC847, Q201 BSS138, Q202 BSS138, Q21 BC847, Q22 DMP3099L, Q23 BC847, Q24 BC847, Q25 DMP3099L, Q26 BC847, Q27 DMP3099L, Q28 DMP3099L, Q29 DMP3099L, Q3 BC847, Q30 DMP3099L, Q31 DMP3099L, Q32 DMP3099L, Q4 BC847, Q5 BC847, Q6 DMP3099L, Q7 BC847, Q8 BC847, Q9 DMP3099L, SW1 RotaryEncoder_Switch, SW2 RotaryEncoder_Switch, U1 TCA9534, U2 TCA9534, U3 TCA9534, U4 uA7805

Commit message: Useless Adder auf V2.0 gebracht. Software finalisiert, Platine benötigt noch Arbeit
Parts:
- D2, D201, D202, D203, D204, D205, D206, D207, D208, D209, D210, D211, D212, D213, D214, D215, D216, D217, D218, D219, D220, D221, D222, D223, D224, D225, D226, D227, D228, D229, D230, D231, D232: footprint Diode_SMD:D_SOD-523 -> Diode_SMD:D_SMF
- D51, D52, D53, D54, D55, D56, D57, D58: footprint Diode_SMD:D_SMF -> Diode_SMD:D_MiniMELF
- Q6: value DMP3099L -> PJM10H01PSA
- moved D226 1.34 mm to (114.5, 206.1)
- moved D206 1.19 mm to (241.1, 155.6)
- moved D2 1.13 mm to (123.2, 96.2)
- moved D217 1.04 mm to (164.3, 193.1)
- moved D214 1.03 mm to (242.0, 168.1)
- moved D222 1.03 mm to (241.0, 193.1)
- moved D207 1.00 mm to (291.9, 155.6)
- moved D216 0.89 mm to (191.0, 168.1)
- moved D201 0.86 mm to (164.3, 155.6)
- moved D204 0.86 mm to (138.9, 155.6)
- moved D215 0.86 mm to (292.5, 168.1)
- moved D211 0.86 mm to (216.4, 168.1)
- moved D212 0.86 mm to (267.0, 168.1)
- moved D220 0.80 mm to (215.5, 193.1)
- moved D213 0.80 mm to (165.5, 168.1)
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Connections:
- K201 pad 11: unconnected-(K201-Pad11) -> +12V
- K201 pad 21: +12V -> unconnected-(K201-Pad21)
- K202 pad 11: Net-(K202-Pad11) -> +12V
- K202 pad 12: unconnected-(K202-Pad12) -> Net-(K202-Pad12)
- K204 pad 11: Net-(K204-Pad11) -> Carry_Bit1_neg
- K204 pad 12: unconnected-(K204-Pad12) -> Net-(K204-Pad12)
- K206 pad 11: Net-(K206-Pad11) -> Carry_Bit2_neg
- K208 pad 11: Net-(K208-Pad11) -> Carry_Bit3_neg
- K208 pad 12: unconnected-(K208-Pad12) -> Net-(K208-Pad12)
- K210 pad 11: Net-(K202-Pad11) -> +12V
- K210 pad 21: unconnected-(K210-Pad21) -> Carry_Bit1_neg
- K210 pad 22: unconnected-(K210-Pad22) -> Net-(K201-Pad12)
- K210 pad 24: unconnected-(K210-Pad24) -> Net-(K202-Pad12)
- K212 pad 11: Net-(K204-Pad11) -> Carry_Bit1_neg
- K212 pad 21: unconnected-(K212-Pad21) -> Carry_Bit2_neg
- K212 pad 22: unconnected-(K212-Pad22) -> Net-(K203-Pad12)
- K212 pad 24: unconnected-(K212-Pad24) -> Net-(K204-Pad12)
- K214 pad 11: Net-(K206-Pad11) -> Carry_Bit2_neg
- K214 pad 21: unconnected-(K214-Pad21) -> Carry_Bit3_neg
- K216 pad 11: Net-(K208-Pad11) -> Carry_Bit3_neg
- K216 pad 21: unconnected-(K216-Pad21) -> Carry_Bit4_neg
- K216 pad 22: unconnected-(K216-Pad22) -> Net-(K207-Pad12)
- K216 pad 24: unconnected-(K216-Pad24) -> Net-(K208-Pad12)
- K218 pad 11: Net-(K218-Pad11) -> Carry_Bit4_neg
- K218 pad 12: unconnected-(K218-Pad12) -> Net-(K218-Pad12)
- K220 pad 11: Net-(K220-Pad11) -> Carry_Bit5_neg
- K220 pad 12: unconnected-(K220-Pad12) -> Net-(K220-Pad12)
- K222 pad 11: Net-(K222-Pad11) -> Carry_Bit6_neg
- K222 pad 12: unconnected-(K222-Pad12) -> Net-(K222-Pad12)
- K224 pad 11: Net-(K224-Pad11) -> Carry_Bit7_neg
- K226 pad 11: Net-(K218-Pad11) -> Carry_Bit4_neg
- K226 pad 21: unconnected-(K226-Pad21) -> Carry_Bit5_neg
- K226 pad 22: unconnected-(K226-Pad22) -> Net-(K217-Pad12)
- K226 pad 24: unconnected-(K226-Pad24) -> Net-(K218-Pad12)
- K228 pad 11: Net-(K220-Pad11) -> Carry_Bit5_neg
- K228 pad 21: unconnected-(K228-Pad21) -> Carry_Bit6_neg
- K228 pad 22: unconnected-(K228-Pad22) -> Net-(K219-Pad12)
- K228 pad 24: unconnected-(K228-Pad24) -> Net-(K220-Pad12)
- K230 pad 11: Net-(K222-Pad11) -> Carry_Bit6_neg
- K230 pad 21: unconnected-(K230-Pad21) -> Carry_Bit7_neg
- K230 pad 22: unconnected-(K230-Pad22) -> Net-(K221-Pad12)
- K230 pad 24: unconnected-(K230-Pad24) -> Net-(K222-Pad12)
- K232 pad 11: Net-(K224-Pad11) -> Carry_Bit7_neg
- SW1 pad MP: GND -> (no net)
- SW2 pad MP: GND -> (no net)
Routing:
- net Carry_Bit4_neg: track 0.00 -> 214.7 mm, vias 0 -> 4
- net GND: track 381.3 -> 263.7 mm
- net Carry_Bit5_neg: track 0.00 -> 97.1 mm
- net Carry_Bit2_neg: track 0.00 -> 97.0 mm, vias 0 -> 2
- net Carry_Bit1_neg: track 0.00 -> 96.8 mm, vias 0 -> 2
- net Carry_Bit3_neg: track 0.00 -> 96.8 mm, vias 0 -> 2
- net Carry_Bit6_neg: track 0.00 -> 96.8 mm
- net Carry_Bit7_neg: track 0.00 -> 96.3 mm
- net +12V: track 783.3 -> 833.8 mm
- net Net-(K208-Pad11): track 38.9 -> 0.00 mm
- net Net-(K222-Pad11): track 38.7 -> 0.00 mm
- net Net-(K202-Pad11): track 38.7 -> 0.00 mm
- net Net-(K220-Pad11): track 38.7 -> 0.00 mm
- net Net-(K218-Pad11): track 38.7 -> 0.00 mm
- net Net-(K206-Pad11): track 38.7 -> 0.00 mm
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Other:
- board text added: "AP 10/2025 Version 2.0"
- board text removed: "AP 09/2025 Version 1.0"

Commit message: DRC durchgeführt und Fehler korrigiert,  Platine verschönert
Routing:
- net GND: track 263.7 -> 380.8 mm, vias 135 -> 145
- net Bit B.4: track 398.8 -> 419.5 mm
- net Bit B.1: track 385.0 -> 404.6 mm
- net Bit B.3: track 395.0 -> 414.6 mm
- net Bit B.2: track 391.2 -> 410.6 mm
- net Bit B.7: track 475.0 -> 489.1 mm
- net Bit B.5: track 465.0 -> 478.8 mm
- net Bit B.6: track 472.8 -> 486.1 mm
- net Bit B.8: track 478.2 -> 491.2 mm
- net Bit A.7: track 310.4 -> 322.9 mm
- net Bit A.8: track 286.8 -> 295.5 mm
- net Bit A.1: track 373.9 -> 382.4 mm
- net Bit A.5: track 416.2 -> 424.6 mm
- net Bit A.2: track 332.0 -> 340.3 mm
- net Bit A.3: track 289.9 -> 298.2 mm
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
Commit message: Umsortiert
Other:
- board text added: "apxco 10/2025 Version 2.0"
- board text removed: "AP 10/2025 Version 2.0"
Changed lines of the file:
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@@
 		)
 	)
-	(gr_text "AP 10/2025\nVersion 2.0"
-		(at 309.118 121.666 0)
+	(gr_text "apxco 10/2025\nVersion 2.0"
+		(at 306.5 120.5 0)
 		(layer "F.SilkS")
 		(effects
