File: Breadboard/OP-V1/OP-V1.kicad_pcb (KiCad board)
At the start: 2 copper layers, 30 parts, among them J1 Conn_01x04_Pin, J2 Conn_01x04_Pin, J4 Conn_01x04_Pin, U1 NE5532, U2 LM311

Commit message: Umsortiert
Other:
- board outline added: 50 x 57 mm
- board text added: "OP Breadboard V2"
- board text removed: "OP Breadboard V1.1"
Changed lines of the file:
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@@
 		(title "OP- Breadboard")
 		(date "2023-11-28")
-		(rev "1.0")
+		(rev "2.0")
 	)
 	(layers
@@
 		(layer "Dwgs.User")
 	)
+	(gr_line
+		(start 191.5 90)
+		(end 241.5 90)
+		(stroke
+			(width 0.1)
+			(type default)
+		)
+		(layer "Edge.Cuts")
+	)
+	(gr_line
+		(start 191.5 147)
+		(end 191.5 90)
+		(stroke
+			(width 0.1)
+			(type default)
+		)
+		(layer "Edge.Cuts")
+	)
+	(gr_line
+		(start 241.5 147)
+		(end 191.5 147)
+		(stroke
+			(width 0.1)
+			(type default)
+		)
+		(layer "Edge.Cuts")
+	)
+	(gr_line
+		(start 191.5 147)
+		(end 191.5 90)
+		(stroke
+			(width 0.15)
+			(type default)
+		)
+		(layer "Margin")
+	)
+	(gr_line
+		(start 191.5 90)
+		(end 241.5 90)
+		(stroke
+			(width 0.15)
+			(type solid)
+		)
+		(layer "Margin")
+	)
+	(gr_line
+		(start 241.5 90)
+		(end 241.5 147)
+		(stroke
+			(width 0.15)
+			(type solid)
+		)
+		(layer "Margin")
+	)
+	(gr_line
+		(start 241.5 147)
+		(end 191.5 147)
+		(stroke
+			(width 0.15)
+			(type default)
+		)
+		(layer "Margin")
+	)
 	(gr_text "GND\n"
 		(at 231.5 143 90)
@@
 		)
 	)
-	(gr_text "OP Breadboard\nV1.1"
+	(gr_text "OP Breadboard\nV2"
 		(at 228.5238 103.3526 0)
 		(layer "F.SilkS")
