File: Netzteile/DCDC_mid/DCDC_mid.kicad_sch (KiCad schematic)
At the start: 37 parts, among them J1 Conn_01x02_Pin, J2 Conn_01x02_Pin, Q1 FTZ953, Q4 Q_PMOS_GDSD, Q5 FTZ853, Q6 FTZ853, U1 TL431LP, U2 LM311

Commit message: Umsortiert
Changed lines of the file:
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@@
 (kicad_sch
-	(version 20231120)
+	(version 20250114)
 	(generator "eeschema")
-	(generator_version "8.0")
+	(generator_version "9.0")
 	(paper "A4")
 	(title_block
@@
 		(comment 3 "P-Kanal Mosfet ")
 	)
+	(text "R6 wird warm"
+		(exclude_from_sim no)
+		(at 92.71 39.37 0)
+		(effects
+			(font
+				(size 1.27 1.27)
+			)
+		)
+	)
+	(text "TL431 Berechnet mit\nUin 20-30V\nUout 13V\n\n"
+		(exclude_from_sim no)
+		(at 30.48 161.925 0)
+		(effects
+			(font
+				(size 1.27 1.27)
+			)
+			(justify left bottom)
+		)
+	)
+	(text "z.B. IRF4905"
+		(exclude_from_sim no)
+		(at 144.78 68.58 0)
+		(effects
+			(font
+				(size 1.27 1.27)
+			)
+		)
+	)
 	(junction
 		(at 102.87 69.85)
@@
 		)
 	)
-	(text "R6 wird warm"
-		(exclude_from_sim no)
-		(at 92.71 39.37 0)
-		(effects
-			(font
-				(size 1.27 1.27)
-			)
-		)
-	)
-	(text "TL431 Berechnet mit\nUin 20-30V\nUout 13V\n\n"
-		(exclude_from_sim no)
-		(at 30.48 161.925 0)
-		(effects
-			(font
-				(size 1.27 1.27)
-			)
-			(justify left bottom)
-		)
-	)
-	(text "z.B. IRF4905"
-		(exclude_from_sim no)
-		(at 144.78 68.58 0)
-		(effects
-			(font
-				(size 1.27 1.27)
-			)
-		)
-	)
 	(symbol
 		(lib_id "Transistor_BJT:BCP56")
@@
 		)
 	)
+	(embedded_fonts no)
 )
