File: Netzteile/Powerbank/Powerbank.kicad_pcb (KiCad board)
At the start: 2 copper layers, 161 x 86 mm, 40 parts, among them J1 Conn_01x04_Female, J2 Conn_01x06_Female

Commit message: Umsortiert
Parts:
- C10, C20, C21, C9: value C_Polarized -> C
Changed lines of the file:
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@@
 			)
 		)
-		(property "Value" "C_Polarized"
+		(property "Value" "C"
 			(at 7.5 3.75 90)
 			(layer "F.Fab")
@@
 			)
 		)
-		(property "Description" ""
+		(property "Description" "Unpolarized capacitor"
 			(at 0 0 90)
 			(layer "F.Fab")
@@
 			)
 		)
-		(property ki_fp_filters "CP_*")
+		(property ki_fp_filters "C_*")
 		(sheetname "/")
 		(sheetfile "Powerbank.kicad_sch")
@@
 			)
 		)
-		(property "Value" "C_Polarized"
+		(property "Value" "C"
 			(at 7.5 3.75 90)
 			(layer "F.Fab")
@@
 			)
 		)
-		(property "Description" ""
+		(property "Description" "Unpolarized capacitor"
 			(at 0 0 90)
 			(layer "F.Fab")
@@
 			)
 		)
-		(property ki_fp_filters "CP_*")
+		(property ki_fp_filters "C_*")
 		(sheetname "/")
 		(sheetfile "Powerbank.kicad_sch")
@@
 			)
 		)
-		(property "Value" "C_Polarized"
+		(property "Value" "C"
 			(at 7.5 3.75 90)
 			(layer "F.Fab")
@@
 			)
 		)
-		(property "Description" ""
+		(property "Description" "Unpolarized capacitor"
 			(at 0 0 90)
 			(layer "F.Fab")
@@
 			)
 		)
-		(property ki_fp_filters "CP_*")
+		(property ki_fp_filters "C_*")
 		(sheetname "/")
 		(sheetfile "Powerbank.kicad_sch")
@@
 			)
 		)
-		(property "Value" "C_Polarized"
+		(property "Value" "C"
 			(at 7.5 3.75 90)
 			(layer "F.Fab")
@@
 			)
 		)
-		(property "Description" ""
+		(property "Description" "Unpolarized capacitor"
 			(at 0 0 90)
 			(layer "F.Fab")
@@
 			)
 		)
-		(property ki_fp_filters "CP_*")
+		(property ki_fp_filters "C_*")
 		(sheetname "/")
 		(sheetfile "Powerbank.kicad_sch")

Commit message: Netzteile überarbeitet, neu sortiert
Parts:
- added C15: C_Polarized, Capacitor_THT:CP_Radial_D10.0mm_P5.00mm_P7.50mm, F.Cu at (177.5, 70.0)
- added C20: C_Polarized, Capacitor_THT:CP_Radial_D10.0mm_P5.00mm_P7.50mm, F.Cu at (177.5, 87.5)
- added C21: C_Polarized, Capacitor_THT:CP_Radial_D10.0mm_P5.00mm_P7.50mm, F.Cu at (107.5, 105.0)
- added C22: C_Polarized, Capacitor_THT:CP_Radial_D10.0mm_P5.00mm_P7.50mm, F.Cu at (125.0, 105.0)
- added C23: C_Polarized, Capacitor_THT:CP_Radial_D10.0mm_P5.00mm_P7.50mm, F.Cu at (142.5, 105.0)
- added C24: C_Polarized, Capacitor_THT:CP_Radial_D10.0mm_P5.00mm_P7.50mm, F.Cu at (160.0, 105.0)
- added C25: C_Polarized, Capacitor_THT:CP_Radial_D10.0mm_P5.00mm_P7.50mm, F.Cu at (177.5, 105.0)
- C10: renamed from C20; value C -> C_Polarized; footprint Capacitor_THT:C_Rect_L16.5mm_W5.0mm_P15.00mm_MKT -> Capacitor_THT:CP_Radial_D10.0mm_P5.00mm_P7.50mm
- C5: renamed from C10; value C -> C_Polarized; footprint Capacitor_THT:C_Rect_L16.5mm_W5.0mm_P15.00mm_MKT -> Capacitor_THT:CP_Radial_D10.0mm_P5.00mm_P7.50mm
- moved C5 86.9 mm to (177.5, 34.5), turned to 90 degrees
- moved C10 73.9 mm to (177.5, 52.0), turned to 90 degrees
- moved C18 16.3 mm to (142.5, 87.5)
- moved C17 16.0 mm to (125.0, 87.5)
- moved C19 16.0 mm to (160.0, 87.5)
- moved C16 15.4 mm to (107.5, 87.5)
- moved C13 14.5 mm to (142.5, 70.0)
- moved C12 14.1 mm to (125.0, 70.0)
- moved C14 14.1 mm to (160.0, 70.0)
- moved C11 13.3 mm to (107.5, 70.0)
- moved C8 12.9 mm to (142.5, 52.5)
- moved C7 12.5 mm to (125.0, 52.5)
- moved C9 12.5 mm to (160.0, 52.5)
- moved H7 12.5 mm to (152.5, 60.0)
- moved C3 11.4 mm to (142.5, 35.0)
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- renumbered C15 to C1, C5 to C11, C19 to C12, C16 to C13, C17 to C14, C18 to C16, C13 to C17, C14 to C18, C3 to C19, C11 to C2, C1 to C26, C9 to C27, C21 to C28, C12 to C3, C2 to C4, C8 to C7, C7 to C8, C4 to C9
Routing:
- net GND: track 450.1 -> 615.0 mm
- net VCC: track 535.9 -> 640.1 mm
- net Net-(D4-A): track 62.1 -> 69.3 mm, vias 0 -> 1
Other:
- board text added: "- A A +"
- board text added: "Netzteil V2 11/2025 apxco"
- board text removed: "Netzteil V2 10/2025 apxco"
