File: Netzteile/Powerbank/Powerbank.kicad_sch (KiCad schematic)
At the start: 40 parts, among them J1 Conn_01x04_Female, J2 Conn_01x06_Female

Commit message: Umsortiert
Parts:
- removed C10, C20, C21, C9: C_Polarized, Capacitor_THT:C_Rect_L16.5mm_W5.0mm_P15.00mm_MKT, symbol Device:C_Polarized
- added C10, C20, C21, C9: C, Capacitor_THT:C_Rect_L16.5mm_W5.0mm_P15.00mm_MKT, symbol Device:C
Connections:
- net GND: now also C10.2, C20.2, C21.2, C9.2
- net VCC: now also C10.1, C20.1, C21.1, C9.1
Other:
- moved on the sheet: C11, C12, C13, C14, C15, C16, C17, C18, C19, C2, C3, C4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

Commit message: Netzteile überarbeitet, neu sortiert
Parts:
- removed C10, C20: C, Capacitor_THT:C_Rect_L16.5mm_W5.0mm_P15.00mm_MKT, symbol Device:C
- added C15, C20, C21, C22, C23, C24, C25, C5, C9: C_Polarized, Capacitor_THT:CP_Radial_D10.0mm_P5.00mm_P7.50mm, symbol Device:C_Polarized
- renumbered C15 to C1, C4 to C10, C5 to C11, C19 to C12, C16 to C13, C17 to C14, C18 to C16, C13 to C17, C14 to C18, C3 to C19, C11 to C2, C1 to C26, C9 to C27, C21 to C28, C12 to C3, C2 to C4, C8 to C7, C7 to C8
Connections:
- net GND: now also C15.2, C20.2, C21.2, C22.2, C23.2, C24.2, C25.2, C5.2, C9.2
- net VCC: now also C15.1, C20.1, C21.1, C22.1, C23.1, C24.1, C25.1, C5.1, C9.1
Other:
- moved on the sheet: C27, C28
