File: Netzteile/Powerbank_2/Powerbank_2.kicad_pcb (KiCad board)
At the start: 2 copper layers, 161 x 86 mm, 40 parts, among them J1 Conn_01x04_Female, J2 Conn_01x06_Female

Commit message: Umsortiert
Parts:
- added C22: C_Polarized, Capacitor_THT:CP_Radial_D10.0mm_P5.00mm_P7.50mm, F.Cu at (175.0, 80.0)
- added C23: C_Polarized, Capacitor_THT:CP_Radial_D10.0mm_P5.00mm_P7.50mm, F.Cu at (175.0, 100.0)
- added D7: LED, LED_THT:LED_D3.0mm_Clear, F.Cu at (90.5, 91.3)
- added F2: Fuse, Fuse:Fuseholder_Littelfuse_100_series_5x20mm, F.Cu at (65.2, 94.6)
- added H10: MountingHole, MountingHole:MountingHole_3.5mm_Pad, F.Cu at (195.0, 32.0)
- added H11: MountingHole, MountingHole:MountingHole_3.5mm_Pad, F.Cu at (195.0, 103.0)
- added R2: R, Resistor_THT:R_Axial_DIN0204_L3.6mm_D1.6mm_P7.62mm_Horizontal, F.Cu at (90.5, 95.2)
- C1: value C_Small -> C_Polarized; footprint Capacitor_THT:C_Axial_L12.0mm_D6.5mm_P15.00mm_Horizontal -> Capacitor_THT:CP_Radial_D10.0mm_P5.00mm_P7.50mm
- C10, C20, C21, C9: footprint Capacitor_THT:C_Rect_L16.5mm_W5.0mm_P15.00mm_MKT -> Capacitor_THT:CP_Radial_D10.0mm_P5.00mm_P7.50mm
- C16, C7: value C_Polarized -> C; footprint Capacitor_THT:CP_Radial_D10.0mm_P5.00mm_P7.50mm -> Capacitor_THT:C_Rect_L16.5mm_W5.0mm_P15.00mm_MKT
- C6: value C_Polarized -> C_Small; footprint Capacitor_THT:CP_Radial_D10.0mm_P5.00mm_P7.50mm -> Capacitor_THT:C_Axial_L12.0mm_D6.5mm_P15.00mm_Horizontal
- D1: value LED -> 1N5408; footprint LED_THT:LED_D3.0mm_Clear -> Diode_THT:D_DO-201AD_P15.24mm_Horizontal
- D3: value 1N5408 -> D_Bridge_-AA+; footprint Diode_THT:D_DO-201AD_P15.24mm_Horizontal -> Diode_THT:Diode_Bridge_Vishay_GBU
- D6: value D_Bridge_-AA+ -> LED; footprint Diode_THT:Diode_Bridge_Vishay_GBU -> LED_THT:LED_D3.0mm_Clear
- H2, H3, H5: value MountingHole -> MountingHole_Pad; footprint MountingHole:MountingHole_3.5mm_Pad -> MountingHole:MountingHole_3.2mm_M3_Pad_TopBottom
- H9: value MountingHole_Pad -> MountingHole; footprint MountingHole:MountingHole_3.2mm_M3_Pad_TopBottom -> MountingHole:MountingHole_3.5mm_Pad
- moved H9 159.9 mm to (51.0, 32.0)
- moved H4 140.1 mm to (195.0, 45.0)
- moved H2 137.6 mm to (50.0, 45.0)
- moved H3 122.4 mm to (64.9, 102.3)
- moved H5 104.2 mm to (184.0, 67.5)
- moved C3 76.1 mm to (130.5, 35.0), turned to -90 degrees
- moved C20 74.5 mm to (145.5, 100.0), turned to 90 degrees
- moved C5 74.0 mm to (175.0, 35.0), turned to -90 degrees
- moved C18 73.8 mm to (175.0, 55.0), turned to -90 degrees
- moved C9 72.0 mm to (115.0, 55.0)
- moved C1 65.6 mm to (115.0, 35.0)
- moved C21 59.9 mm to (130.5, 100.0), turned to 90 degrees
- moved C16 59.1 mm to (99.0, 103.9)
- moved C7 55.5 mm to (99.0, 47.2)
- moved H1 55.2 mm to (64.9, 35.7)
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Connections:
- C1 pad 1: Net-(D4-A) -> VCC
- C1 pad 2: Net-(D2-A) -> GND
- C12 pad 1: VCC -> GND
- C12 pad 2: GND -> VPP
- C13 pad 1: VCC -> GND
- C13 pad 2: GND -> VPP
- C14 pad 1: VCC -> GND
- C14 pad 2: GND -> VPP
- C15 pad 1: VCC -> GND
- C15 pad 2: GND -> VPP
- C16 pad 1: VCC -> GND
- C16 pad 2: GND -> VPP
- C17 pad 1: VCC -> GND
- C17 pad 2: GND -> VPP
- C19 pad 1: VCC -> GND
- C19 pad 2: GND -> VPP
- C20 pad 1: VCC -> GND
- C20 pad 2: GND -> VPP
- C21 pad 1: VCC -> GND
- C21 pad 2: GND -> VPP
- C6 pad 1: VCC -> Net-(D2-A)
- C6 pad 2: GND -> Net-(D1-A)
- D1 pad 1: Net-(D1-K) -> VCC
- D1 pad 2: VCC -> Net-(D1-A)
- D3 pad 1: Net-(D2-A) -> VPP
- D3 pad 2: GND -> Net-(D2-A)
- D4 pad 1: VCC -> Net-(D1-A)
- D4 pad 2: Net-(D4-A) -> VPP
- D5 pad 1: Net-(D4-A) -> Net-(D2-A)
- D5 pad 2: GND -> VPP
- D6 pad 1: GND -> Net-(D6-K)
- D6 pad 2: Net-(D4-A) -> VCC
- F1 pad 1: Net-(J1-Pin_3) -> Net-(J1-Pin_4)
- F1 pad 2: Net-(D4-A) -> Net-(D2-A)
- H1 pad 1: Net-(D2-A) -> Net-(J1-Pin_4)
- H2 pad 1: (no net) -> GND
- H3 pad 1: (no net) -> Net-(J1-Pin_1)
- H4 pad 1: Net-(J1-Pin_3) -> VCC
- H5 pad 1: (no net) -> GND
- H8 pad 1: VCC -> VPP
- H9 pad 1: GND -> (no net)
- J1 pad 1: Net-(D2-A) -> Net-(J1-Pin_1)
- J1 pad 2: Net-(D2-A) -> GND
- J1 pad 3: Net-(J1-Pin_3) -> GND
- J1 pad 4: Net-(J1-Pin_3) -> Net-(J1-Pin_4)
- J2 pad 1: VCC -> VPP
- J2 pad 2: VCC -> VPP
- J2 pad 3: VCC -> GND
- J2 pad 5: GND -> VCC
- J2 pad 6: GND -> VCC
- R1 pad 1: Net-(D1-K) -> Net-(D6-K)
Routing:
- net VPP: track 0.00 -> 331.2 mm
- net VCC: track 535.9 -> 323.7 mm
- net GND: track 450.1 -> 370.5 mm, vias 21 -> 14
- net Net-(D4-A): track 62.1 -> 0.00 mm
- net Net-(D1-A): track 0.00 -> 60.5 mm
- net Net-(J1-Pin_3): track 39.7 -> 0.00 mm
- net Net-(J1-Pin_1): track 0.00 -> 32.6 mm
- net Net-(J1-Pin_4): track 0.00 -> 30.9 mm
- net Net-(D2-A): track 86.7 -> 98.1 mm
- net Net-(D6-K): track 0.00 -> 5.53 mm
- net Net-(D1-K): track 5.00 -> 0.00 mm
- net Net-(D7-K): track 0.00 -> 3.87 mm
- added copper zone on F.Cu, net VPP
Other:
- board text added: "GND"
- board text added: "Negativ"
- board text added: "Netzteil V3 11/2025 apxco"
- board text removed: "Negativ (GND)"
- board text removed: "Netzteil V2 10/2025 apxco"

Commit message: Netzteile überarbeitet, neu sortiert
Parts:
- added C11: C_Polarized, Capacitor_THT:CP_Radial_D10.0mm_P5.00mm_P7.50mm, F.Cu at (114.5, 58.8)
- added C12: C_Polarized, Capacitor_THT:CP_Radial_D10.0mm_P5.00mm_P7.50mm, F.Cu at (130.0, 58.8)
- added C13: C_Polarized, Capacitor_THT:CP_Radial_D10.0mm_P5.00mm_P7.50mm, F.Cu at (145.0, 58.8)
- added C14: C_Polarized, Capacitor_THT:CP_Radial_D10.0mm_P5.00mm_P7.50mm, F.Cu at (160.0, 58.8)
- added C15: C_Polarized, Capacitor_THT:CP_Radial_D10.0mm_P5.00mm_P7.50mm, F.Cu at (174.5, 58.8)
- added C16: C_Polarized, Capacitor_THT:CP_Radial_D10.0mm_P5.00mm_P7.50mm, F.Cu at (114.5, 77.5)
- added C17: C_Polarized, Capacitor_THT:CP_Radial_D10.0mm_P5.00mm_P7.50mm, F.Cu at (130.0, 77.5)
- added C18: C_Polarized, Capacitor_THT:CP_Radial_D10.0mm_P5.00mm_P7.50mm, F.Cu at (145.0, 77.5)
- added C19: C_Polarized, Capacitor_THT:CP_Radial_D10.0mm_P5.00mm_P7.50mm, F.Cu at (160.0, 77.5)
- added C20: C_Polarized, Capacitor_THT:CP_Radial_D10.0mm_P5.00mm_P7.50mm, F.Cu at (174.5, 77.5)
- moved C21 12.5 mm to (115.0, 92.5)
- moved C22 12.5 mm to (130.5, 92.5)
- moved C23 12.5 mm to (145.5, 92.5)
- moved C24 12.5 mm to (160.5, 92.5)
- moved C25 12.5 mm to (175.0, 92.5)
- moved C10 10.7 mm to (175.0, 44.3)
- moved C6 10.7 mm to (115.0, 44.3)
- moved C7 10.7 mm to (130.5, 44.3)
- moved C8 10.7 mm to (145.5, 44.3)
- moved C9 10.7 mm to (160.5, 44.3)
- moved H7 10.0 mm to (152.5, 67.5)
- moved C26 5.00 mm to (115.0, 105.0)
- moved C27 5.00 mm to (130.5, 105.0)
- moved C28 5.00 mm to (145.5, 105.0)
- moved C29 5.00 mm to (160.5, 105.0)
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- renumbered C18 to C10, C3 to C2, C14 to C21, C15 to C22, C13 to C23, C12 to C24, C22 to C25, C19 to C26, C21 to C27, C20 to C28, C17 to C29, C4 to C3, C23 to C30, C6 to C31, C7 to C32, C16 to C33, C2 to C4, C9 to C6, C11 to C7, C10 to C8, C8 to C9
Routing:
- net GND: track 370.5 -> 42.3 mm, vias 14 -> 15
- net VPP: track 331.2 -> 406.8 mm
- net VCC: track 323.7 -> 392.4 mm
Other:
- board text added: "- A A +"
