File: Netzteile/Powerbank_2/Powerbank_2.kicad_sch (KiCad schematic)
At the start: 40 parts, among them J1 Conn_01x04_Female, J2 Conn_01x06_Female

Commit message: Umsortiert
Parts:
- removed C10, C20, C21, C9: C_Polarized, Capacitor_THT:C_Rect_L16.5mm_W5.0mm_P15.00mm_MKT, symbol Device:C_Polarized
- added C16, C7: C, Capacitor_THT:C_Rect_L16.5mm_W5.0mm_P15.00mm_MKT, symbol Device:C
- added C18, C22, C23, C5: C_Polarized, Capacitor_THT:CP_Radial_D10.0mm_P5.00mm_P7.50mm, symbol Device:C_Polarized
- added D7: LED, LED_THT:LED_D3.0mm_Clear, symbol Device:LED
- added F2: Fuse, Fuse:Fuseholder_Littelfuse_100_series_5x20mm, symbol Device:Fuse
- added H2, H5: MountingHole_Pad, MountingHole:MountingHole_3.2mm_M3_Pad_TopBottom, symbol Mechanical:MountingHole_Pad
- added R2: R, Resistor_THT:R_Axial_DIN0204_L3.6mm_D1.6mm_P7.62mm_Horizontal, symbol Device:R
- renumbered C15 to C1, C7 to C10, C8 to C11, C17 to C12, C16 to C13, C5 to C14, C19 to C15, C3 to C17, C18 to C19, C14 to C20, C13 to C21, C11 to C3, C12 to C4, C1 to C6, C4 to C8, C6 to C9, D2 to D1, D4 to D2, D6 to D3, D3 to D4, D1 to D6, H4 to H1, H6 to H10, H7 to H11, H1 to H3, H8 to H4, H2 to H6, H5 to H7, H9 to H8, H3 to H9
Connections:
- net GND: now also C12.1, C13.1, C14.1, C15.1, C17.1, C19.1, C20.1, C21.1, J1.2 (Pin_2), J1.3 (Pin_3), J2.3 (Pin_3), C16.1, C18.2, C22.1, C23.1, C5.2, C7.2, D7.2 (A), H2.1, H5.1; no longer C12.2, C13.2, C14.2, C15.2, C17.2, C19.2, C20.2, C21.2, D3.1 (-), D4.2 (A), D5.2 (A), H8.1, J2.5 (Pin_5), J2.6 (Pin_6)
- net VCC: now also J2.5 (Pin_5), J2.6 (Pin_6), C18.1, C5.1, C7.1; no longer C12.1, C13.1, C14.1, C15.1, C17.1, C19.1, C20.1, C21.1, J2.1 (Pin_1), J2.2 (Pin_2), J2.3 (Pin_3)
- net at C6.2, D1.2 (A), D3.3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: now also F2.2; no longer H3.1, J1.1 (Pin_1), J1.2 (Pin_2)
- net at F1.1, H1.1, J1.4 (Pin_4): no longer J1.3 (Pin_3)
- new net: F2.1, H3.1, J1.1 (Pin_1)
- new net: D7.1 (K), R2.1
- new net VPP: C12.2, C13.2, C14.2, C15.2, C16.2, C17.2, C19.2, C20.2, C21.2, C22.2, C23.2, D3.1 (-), D4.2 (A), D5.2 (A), H8.1, J2.1 (Pin_1), J2.2 (Pin_2), R2.2
Other:
- title: Netzteilplatine -> Netzteilplatine für Duale Spannungsversorgung
- moved on the sheet: C1, C10, C11, C12, C13, C14, C15, C17, C19, C2, C20, C21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

Commit message: Netzteile überarbeitet, neu sortiert
Parts:
- removed C2: C_Polarized, Capacitor_THT:CP_Radial_D10.0mm_P5.00mm_P7.50mm, symbol Device:C_Polarized
- added C16, C24, C25, C26, C27, C28, C29, C3, C30, C6, C7: C_Polarized, Capacitor_THT:CP_Radial_D10.0mm_P5.00mm_P7.50mm, symbol Device:C_Polarized
- renumbered C3 to C2, C6 to C31, C7 to C32, C16 to C33
Connections:
- net GND: now also C12.2, C13.2, C14.2, C15.2, C18.1, C16.1, C24.1, C25.1, C26.1, C27.1, C28.1, C29.1, C3.2, C30.1, C6.2, C7.2; no longer C12.1, C13.1, C14.1, C15.1, C18.2
- net VCC: now also C12.1, C13.1, C14.1, C15.1, C3.1, C6.1, C7.1; no longer C18.1
- net VPP: now also C18.2, C16.2, C24.2, C25.2, C26.2, C27.2, C28.2, C29.2, C30.2; no longer C12.2, C13.2, C14.2, C15.2
Other:
- moved on the sheet: C2, C32, H10, H11, H7
