File: Useless_Relais_Adder/RelaisAddierer/RelaisAddierer.kicad_pcb (KiCad board)
At the start: 2 copper layers, 290.1 x 175 mm, 254 parts, among them J1 Conn_01x08_Pin, J2 Barrel_Jack, K201 HK19F-DCxxV-SHC, K202 HK19F-DCxxV-SHC, K203 HK19F-DCxxV-SHC, K204 HK19F-DCxxV-SHC, K205 HK19F-DCxxV-SHC, K206 HK19F-DCxxV-SHC, K207 HK19F-DCxxV-SHC, K208 HK19F-DCxxV-SHC, K209 HK19F-DCxxV-SHC, K210 HK19F-DCxxV-SHC, K211 HK19F-DCxxV-SHC, K212 HK19F-DCxxV-SHC, K213 HK19F-DCxxV-SHC, K214 HK19F-DCxxV-SHC, K215 HK19F-DCxxV-SHC, K216 HK19F-DCxxV-SHC, K217 HK19F-DCxxV-SHC, K218 HK19F-DCxxV-SHC, K219 HK19F-DCxxV-SHC, K220 HK19F-DCxxV-SHC, K221 HK19F-DCxxV-SHC, K222 HK19F-DCxxV-SHC, K223 HK19F-DCxxV-SHC, K224 HK19F-DCxxV-SHC, K225 HK19F-DCxxV-SHC, K226 HK19F-DCxxV-SHC, K227 HK19F-DCxxV-SHC, K228 HK19F-DCxxV-SHC, K229 HK19F-DCxxV-SHC, K230 HK19F-DCxxV-SHC, K231 HK19F-DCxxV-SHC, K232 HK19F-DCxxV-SHC, Q1 BC847, Q10 BC847, Q11 DMP3099L, Q12 DMP3099L, Q13 DMP3099L, Q14 DMP3099L, Q15 DMP3099L, Q16 DMP3099L, Q17 BC847, Q18 BC847, Q19 BC847, Q2 BC847, Q20 BC847, Q201 BSS138, Q202 BSS138, Q21 BC847, Q22 DMP3099L, Q23 BC847, Q24 BC847, Q25 DMP3099L, Q26 BC847, Q27 DMP3099L, Q28 DMP3099L, Q29 DMP3099L, Q3 BC847, Q30 DMP3099L, Q31 DMP3099L, Q32 DMP3099L, Q4 BC847, Q5 BC847, Q6 PJM10H01PSA, Q7 BC847, Q8 BC847, Q9 DMP3099L, SW1 RotaryEncoder_Switch, SW2 RotaryEncoder_Switch, U1 TCA9534, U2 TCA9534, U3 TCA9534, U4 uA7805

Commit message: Spannungsteiler statt Widerstand für Eingangsstufe
Parts:
- added R10: 1k, Resistor_SMD:R_0805_2012Metric_Pad1.20x1.40mm_HandSolder, F.Cu at (163.9, 126.0)
- added R7: 1k, Resistor_SMD:R_0805_2012Metric_Pad1.20x1.40mm_HandSolder, F.Cu at (163.9, 137.0)
- added R8: 1k, Resistor_SMD:R_0805_2012Metric_Pad1.20x1.40mm_HandSolder, F.Cu at (163.9, 133.5)
- added R9: 1k, Resistor_SMD:R_0805_2012Metric_Pad1.20x1.40mm_HandSolder, F.Cu at (163.9, 129.5)
- added R93: 1k, Resistor_SMD:R_0805_2012Metric_Pad1.20x1.40mm_HandSolder, F.Cu at (163.9, 122.0)
- added R94: 1k, Resistor_SMD:R_0805_2012Metric_Pad1.20x1.40mm_HandSolder, F.Cu at (163.9, 118.0)
- added R95: 1k, Resistor_SMD:R_0805_2012Metric_Pad1.20x1.40mm_HandSolder, F.Cu at (163.9, 114.5)
- added R96: 1k, Resistor_SMD:R_0805_2012Metric_Pad1.20x1.40mm_HandSolder, F.Cu at (163.9, 111.0)
- R76, R77, R78, R79, R80, R81, R82: value 560 -> 1k
- moved D57 3.66 mm to (172.2, 126.0)
- moved D54 3.66 mm to (172.2, 114.5)
- moved D53 3.65 mm to (172.2, 133.5)
- moved D51 3.65 mm to (172.1, 137.0)
- moved D56 3.65 mm to (172.2, 118.0)
- moved D52 3.65 mm to (172.2, 111.0)
- moved D58 3.65 mm to (172.2, 121.9)
- moved D55 3.65 mm to (172.2, 129.5)
- moved R76 2.62 mm to (177.4, 136.9)
- moved R82 2.57 mm to (177.4, 126.0)
- moved R79 2.57 mm to (177.4, 114.5)
- moved R78 2.56 mm to (177.4, 133.5)
- moved R81 2.55 mm to (177.4, 118.0)
- moved R77 2.55 mm to (177.4, 111.0)
- moved R80 2.55 mm to (177.4, 129.5)
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Routing:
- net GND: track 380.8 -> 393.2 mm, vias 145 -> 153
- net Net-(D51-K): track 33.6 -> 42.8 mm
- net Net-(D53-K): track 30.8 -> 38.8 mm
- net Net-(D58-K): track 25.5 -> 31.9 mm
- net Net-(D55-K): track 28.2 -> 34.5 mm
- net Net-(D57-K): track 25.7 -> 30.6 mm
- net Net-(D52-K): track 23.5 -> 28.2 mm
- net Net-(D54-K): track 23.5 -> 28.0 mm
- net Net-(D56-K): track 24.8 -> 29.1 mm
- net Summ_Bit4: track 215.6 -> 212.9 mm
- net Summ_Bit5: track 239.2 -> 236.5 mm
- net Summ_Bit3: track 165.5 -> 162.9 mm
- net Summ_Bit2: track 115.7 -> 113.1 mm
- net Summ_Bit8: track 389.6 -> 387.1 mm
- net Summ_Bit6: track 290.2 -> 287.7 mm
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