File: Useless_Relais_Adder2/RelaisAdderII.kicad_pcb (KiCad board)
At the start: 2 copper layers, 195 x 105 mm, 164 parts, among them J1 Conn_01x08_Pin, J2 USB_C_Receptacle_PowerOnly_6P, K2 HK19F-DCxxV-SHC, K3 HK19F-DCxxV-SHC, K4 HK19F-DCxxV-SHC, K5 HK19F-DCxxV-SHC, Q10 BC847, Q2 PJM10H01PSA, Q3 DMP3099L, Q4 BC847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

Commit message: Version 1.0 für Platinenherstellung
Parts:
- moved J2 12.0 mm to (90.0, 122.0)
- moved R70 12.0 mm to (91.0, 133.5)
- moved R71 12.0 mm to (91.0, 130.5)
- moved H2 10.0 mm to (95.0, 56.0)
- moved H4 10.0 mm to (95.0, 151.0)
- moved R50 5.02 mm to (95.0, 91.6)
- moved R68 5.02 mm to (95.0, 94.0)
- moved C7 0.98 mm to (143.7, 110.3)
Connections:
- A2 pad 10: SRCLK -> SRCLK_Cary
- A2 pad 11: SCLR_Cary -> RCLK
- A2 pad 12: RCLK -> SCLR_Cary
- A2 pad 13: unconnected-(A2-D10-Pad13) -> SRCLK
- A2 pad 5: Net-(A2-D2) -> unconnected-(A2-D2-Pad5)
- A2 pad 6: Net-(A2-D3) -> SCLR
- A2 pad 7: SCLR -> Net-(A2-D4)
- A2 pad 8: RCLK_Cary -> Net-(A2-D5)
- A2 pad 9: SRCLK_Cary -> RCLK_Cary
- R50 pad 2: Net-(A2-D2) -> Net-(A2-D4)
- R68 pad 2: Net-(A2-D3) -> Net-(A2-D5)
Routing:
- net SCLR: track 332.0 -> 279.9 mm
- net A_Ausg: track 320.7 -> 283.6 mm, vias 4 -> 2
- net +5V: track 584.7 -> 571.3 mm, vias 24 -> 22
- net B_Ausg: track 296.4 -> 287.7 mm, vias 0 -> 2
- net Net-(A2-D3): track 5.27 -> 0.00 mm
- net Net-(A2-D2): track 5.17 -> 0.00 mm
- net RCLK: track 291.5 -> 286.4 mm
- net Net-(A2-D5): track 0.00 -> 4.93 mm
- net Net-(A2-D4): track 0.00 -> 4.90 mm
- net SRCLK: track 295.2 -> 298.7 mm, vias 7 -> 8
- net Summ: track 173.1 -> 176.6 mm
- net SCLR_Cary: track 58.4 -> 55.9 mm
- net SRCLK_Cary: track 62.2 -> 60.1 mm
- net Carry: track 142.8 -> 144.5 mm
- net RCLK_Cary: track 63.0 -> 61.9 mm
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Other:
- board size 195 x 105 mm -> 183.2 x 105 mm
- board text added: "Useless Relais Adder II V1.0 02/2026 apxco"
