File: Useless_Relais_Adder2/RelaisAdderII.kicad_sch (KiCad schematic)
At the start: 164 parts, among them J1 Conn_01x08_Pin, J2 USB_C_Receptacle_PowerOnly_6P, K2 HK19F-DCxxV-SHC, K3 HK19F-DCxxV-SHC, K4 HK19F-DCxxV-SHC, K5 HK19F-DCxxV-SHC, Q10 BC847, Q2 PJM10H01PSA, Q3 DMP3099L, Q4 BC847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

Commit message: Version 1.0 für Platinenherstellung
Connections:
- net RCLK: now also A2.11 (D8); no longer A2.12 (D9)
- net RCLK_Cary: now also A2.9 (D6); no longer A2.8 (D5)
- net SCLR: now also A2.6 (D3); no longer A2.7 (D4)
- net SCLR_Cary: now also A2.12 (D9); no longer A2.11 (D8)
- net SRCLK: now also A2.13 (D10); no longer A2.10 (D7)
- net SRCLK_Cary: now also A2.10 (D7); no longer A2.9 (D6)
- net at R68.2: now also A2.8 (D5); no longer A2.6 (D3)
- net at R50.2: now also A2.7 (D4); no longer A2.5 (D2)
- no-connect marks 1 -> 22
Other:
- moved on the sheet: R50, R68
